Commit message: Merge branch 'gears' into hydro-devel

File: pandora_models/pandora_sensors_description/urdf/co2_sensor.urdf.xacro (robot description, xacro)
@@ -1,51 +1,61 @@
 <?xml version="1.0" ?>
-<robot xmlns:xacro="http://ros.org/wiki/xacro">
-<xacro:macro name="co2_caster" params="parent *origin">
-      <link name="co2_link">
+<robot xmlns:xacro="http://ros.org/wiki/xacro" >
+  <xacro:macro name="co2_caster"
+               params="parent *origin" >
+    <link name="co2_link" >
       <inertial>
-      <mass value="0.1"/>
-      <origin xyz="0 0 0"/>
-      <inertia ixx="0.0001" ixy="0" ixz="0" iyy="0.0001" iyz="0" izz="0.0001" />
+        <mass value="0.1" />
+        <origin xyz="0 0 0" />
+        <inertia ixx="1"
+                 ixy="0"
+                 ixz="0"
+                 iyy="1"
+                 iyz="0"
+                 izz="1" />
       </inertial>
-        <visual name="visual">
-      <origin xyz="0 0 0" rpy="0 0 0"/>
-          <geometry>
-      <mesh filename="package://pandora_sensors_description/meshes/co2_sensor/co2_small.dae"/>
-          </geometry>
-        </visual>
-        <collision name="collision">
-      <origin xyz="0 0 0" rpy="0 0 0"/>
-          <geometry>
-            <box size="0.01 0.01 0.01"/>
-          </geometry>
-        </collision>
+      <visual name="visual" >
+        <origin xyz="0 0 0"
+                rpy="0 0 0" />
+        <geometry>
+          <mesh filename="package://pandora_sensors_description/meshes/co2_sensor/co2_small.dae" />
+        </geometry>
+      </visual>
+      <collision name="collision" >
+        <origin xyz="0 0 0"
+                rpy="0 0 0" />
+        <geometry>
+          <box size="0.01 0.01 0.01" />
+        </geometry>
+      </collision>
     </link>
-    <gazebo reference="co2_link">
-    <sensor name="co2" type="camera">
-      <camera>
-        <horizontal_fov>1.5</horizontal_fov>
-        <image>
-          <width>640</width>
-          <height>480</height>
-        </image>
-        <clip>
-          <near>0.1</near>
-          <far>0.8</far>
-        </clip>
-      </camera>
-      <always_on>1</always_on>
-      <update_rate>5</update_rate>
-      <visualize>false</visualize>
-      <plugin name="co2ros" filename="libpandora_co2_plugin.so">
-        <frameName>co2</frameName>
-        <topicName>sensors/co2</topicName>
-      </plugin>
-    </sensor>
-  </gazebo>
-  <joint name="co2_joint" type="fixed">
-    <xacro:insert_block name="origin" />
-    <parent link="${parent}"/>
-    <child link="co2_link"/>
-  </joint>
-</xacro:macro>
+    <gazebo reference="co2_link" >
+      <sensor name="co2" type="camera" >
+        <camera>
+          <horizontal_fov>1.5</horizontal_fov>
+          <image>
+            <width>640</width>
+            <height>480</height>
+          </image>
+          <clip>
+            <near>0.1</near>
+            <far>0.8</far>
+          </clip>
+        </camera>
+        <always_on>1</always_on>
+        <update_rate>5</update_rate>
+        <visualize>false</visualize>
+        <plugin name="co2ros"
+                filename="libpandora_co2_plugin.so" >
+          <frameName>co2</frameName>
+          <topicName>sensors/co2</topicName>
+        </plugin>
+      </sensor>
+    </gazebo>
+    <joint name="co2_joint"
+           type="fixed" >
+      <parent link="${parent}" />
+      <child link="co2_link" />
+      <xacro:insert_block name="origin" />
+    </joint>
+  </xacro:macro>
 </robot>

File: pandora_models/pandora_sensors_description/urdf/microphone_sensor.urdf.xacro (robot description, xacro)
@@ -1,51 +1,61 @@
 <?xml version="1.0" ?>
-<robot xmlns:xacro="http://ros.org/wiki/xacro">
-<xacro:macro name="microphone_caster" params="parent *origin">
-  <link name="microphone_link">
-    <inertial>
-      <mass value="0.1"/>
-      <origin xyz="0 0 0"/>
-      <inertia ixx="0.0001" ixy="0" ixz="0" iyy="0.0001" iyz="0" izz="0.0001" />
-    </inertial>
-    <visual name="visual">
-      <origin xyz="0 0 0" rpy="0 0 0"/>
-      <geometry>
-        <mesh filename="package://pandora_sensors_description/meshes/microphone_sensor/microphone_small.dae"/>
-      </geometry>
-    </visual>
-    <collision name="collision">
-      <origin xyz="0 0 0" rpy="0 0 0"/>
-      <geometry>
-        <box size="0.01 0.01 0.01"/>
-      </geometry>
-    </collision>
-  </link>
-  <gazebo reference="microphone_link">
-    <sensor name="microphone" type="camera">
-      <camera>
-        <horizontal_fov>1.5</horizontal_fov>
-        <image>
-          <width>640</width>
-          <height>480</height>
-        </image>
-        <clip>
-          <near>0.1</near>
-          <far>2</far>
-        </clip>
-      </camera>
-      <always_on>1</always_on>
-      <update_rate>10</update_rate>
-      <visualize>false</visualize>
-      <plugin name="microphone2ros" filename="libpandora_microphone_plugin.so">
-        <frameName>sound</frameName>
-        <topicName>sensors/sound</topicName>
-      </plugin>
-    </sensor>
-  </gazebo>
-  <joint name="microphone_joint" type="fixed">
-    <xacro:insert_block name="origin" />
-      <parent link="${parent}"/>
-    <child link="microphone_link"/>
-  </joint>
-</xacro:macro>
+<robot xmlns:xacro="http://ros.org/wiki/xacro" >
+  <xacro:macro name="microphone_caster"
+               params="parent *origin" >
+    <link name="microphone_link" >
+      <inertial>
+        <mass value="0.1" />
+        <origin xyz="0 0 0" />
+        <inertia ixx="1"
+                 ixy="0"
+                 ixz="0"
+                 iyy="1"
+                 iyz="0"
+                 izz="1" />
+      </inertial>
+      <visual name="visual" >
+        <origin xyz="0 0 0"
+                rpy="0 0 0" />
+        <geometry>
+          <mesh filename="package://pandora_sensors_description/meshes/microphone_sensor/microphone_small.dae" />
+        </geometry>
+      </visual>
+      <collision name="collision" >
+        <origin xyz="0 0 0"
+                rpy="0 0 0" />
+        <geometry>
+          <box size="0.01 0.01 0.01" />
+        </geometry>
+      </collision>
+    </link>
+    <gazebo reference="microphone_link" >
+      <sensor name="microphone"
+              type="camera" >
+        <camera>
+          <horizontal_fov>1.5</horizontal_fov>
+          <image>
+            <width>640</width>
+            <height>480</height>
+          </image>
+          <clip>
+            <near>0.1</near>
+            <far>2</far>
+          </clip>
+        </camera>
+        <always_on>1</always_on>
+        <update_rate>10</update_rate>
+        <visualize>false</visualize>
+        <plugin name="microphone2ros"
+                filename="libpandora_microphone_plugin.so" >
+          <frameName>sound</frameName>
+          <topicName>sensors/sound</topicName>
+        </plugin>
+      </sensor>
+    </gazebo>
+    <joint name="microphone_joint" type="fixed" >
+      <xacro:insert_block name="origin" />
+      <parent link="${parent}" />
+      <child link="microphone_link" />
+    </joint>
+  </xacro:macro>
 </robot>

File: pandora_models/pandora_sensors_description/urdf/thermal_sensor.urdf.xacro (robot description, xacro)
@@ -1,34 +1,41 @@
 <?xml version="1.0" ?>
-<robot xmlns:xacro="http://ros.org/wiki/xacro">
-<xacro:macro name="thermal_caster" params="parent *origin">
-    <link name="thermal_link">
+<robot xmlns:xacro="http://ros.org/wiki/xacro" >
+  <xacro:macro name="thermal_caster"
+               params="parent *origin" >
+    <link name="thermal_link" >
       <inertial>
-        <origin xyz="0 0 0.186" rpy="0 0 0"/>
-        <mass value="0.1"/>
-        <inertia ixx="0.0001" ixy="0.0" ixz="0.0"
-             iyy="0.0001" iyz="0.0" izz="0.0001"/>
+        <origin xyz="0 0 0.186"
+                rpy="0 0 0" />
+        <mass value="0.1" />
+        <inertia ixx="1.0"
+                 ixy="0.0"
+                 ixz="0.0"
+                 iyy="1.0"
+                 iyz="0.0"
+                 izz="1.0" />
       </inertial>
-      <visual name="visual">
+      <visual name="visual" >
         <geometry>
-         <mesh filename="package://pandora_sensors_description/meshes/thermal_sensor/thermal_small.dae"/>
+          <mesh filename="package://pandora_sensors_description/meshes/thermal_sensor/thermal_small.dae" />
         </geometry>
       </visual>
-      <collision name="collision">
+      <collision name="collision" >
         <geometry>
-          <box size="0.01 0.01 0.01"/>
+          <box size="0.01 0.01 0.01" />
         </geometry>
       </collision>
     </link>
-    <gazebo reference="thermal_link">
-    <sensor name="thermal" type="camera">
+    <gazebo reference="thermal_link" >
+      <sensor name="thermal"
+              type="camera" >
         <camera>
-          <horizontal_fov>0.5</horizontal_fov>
+          <horizontal_fov>0.8</horizontal_fov>
           <image>
-            <width>8</width>
-            <height>8</height>
+            <width>640</width>
+            <height>480</height>
           </image>
           <clip>
-            <near>0.1</near>
-            <far>2</far>
+            <near>0.05</near>
+            <far>1.5</far>
           </clip>
         </camera>
@@ -36,15 +43,17 @@
         <update_rate>30</update_rate>
         <visualize>false</visualize>
-        <plugin name="thermal2ros" filename="libpandora_thermal_plugin.so">
-        <frameName>thermal_link</frameName>
-        <topicName>sensors/thermal</topicName>
-      </plugin>
+        <plugin name="thermal2ros"
+                filename="libpandora_thermal_plugin.so" >
+          <frameName>thermal_link</frameName>
+          <topicName>sensors/thermal</topicName>
+        </plugin>
       </sensor>
-  </gazebo>
-  <joint name="thermal_joint" type="fixed">
-    <xacro:insert_block name="origin" />
-      <parent link="${parent}"/>
-    <child link="thermal_link"/>
-  </joint>
-</xacro:macro>
+    </gazebo>
+    <joint name="thermal_joint"
+           type="fixed" >
+      <parent link="${parent}" />
+      <child link="thermal_link" />
+      <xacro:insert_block name="origin" />
+    </joint>
+  </xacro:macro>
 </robot>
