Commit message: Fix kinect_platform origin

File: pandora_models/pandora_sensors_description/urdf/kinect.urdf.xacro (robot description, xacro)
@@ -115,6 +115,4 @@
         <parent link="kinect_pitch_servo_link" />
         <child link="kinect_platform_link" />
-        <origin xyz="0.0 0.0 0.02852"
-                rpy="0.0 0.0 0.0" />
       </joint>
     </xacro:if>
@@ -136,6 +134,4 @@
         <parent link="kinect_pitch_servo_link" />
         <child link="kinect_platform_link" />
-        <origin xyz="0.0 0.0 0.02852"
-                rpy="0.0 0.0 0.0" />
         <axis xyz="0 1 0" />
         <limit lower="${pitch_min_limit}"
@@ -149,5 +145,5 @@
       <parent link="kinect_platform_link" />
       <child link="kinect_link" />
-      <origin xyz="0.03261 -0.00101 0.01409"
+      <origin xyz="0.03261 -0.00101 0.04261"
               rpy="0.0 0.0 0.0" />
     </joint>
