Commit message: Add cameras to urdf.

File: pandora_models/pandora_robots_description/urdf/gears/sensors/kinect_sensor.xacro (robot description, xacro)
@@ -13,6 +13,6 @@
                          yaw_min_limit="${kinect_yaw_joint_min_limit}"
                          yaw_max_limit="${kinect_yaw_joint_max_limit}" >
-      <origin xyz="0.06744 0.01239 0.19742"
-              rpy="${zero}" />
+      <origin xyz="0.07044 0.01239 0.14642"
+              rpy="-0.0436 0.0 0.0" />
     </xacro:kinect_caster>
   </xacro:macro>

File: pandora_models/pandora_robots_description/urdf/gears/sensors/laser_sensor.xacro (robot description, xacro)
@@ -13,5 +13,5 @@
                          pitch_min_limit="${laser_pitch_joint_min_limit}"
                          pitch_max_limit="${laser_pitch_joint_max_limit}" >
-      <origin xyz="0.1894 0.0 0.09679"
+      <origin xyz="0.1974 0.0 0.09679"
               rpy="${zero}" />
     </xacro:hokuyo_caster>
