Commit message: Update sensor meshes and fix their positions.

File: pandora_models/pandora_robots_description/urdf/gears/links/wheel_link.urdf.xacro (robot description, xacro)
@@ -9,12 +9,12 @@
         <origin xyz="${ reflect_y * ( -2.2235E-05 ) } ${ reflect_y * ( -0.00052624 ) } 2.4287E-05" />
         <!-- ============================================================== -->
-        <mass value="6.90375" />
+        <mass value="1.5" />
         <!-- ============================================================== -->
-        <inertia ixx="0.0201150"
-                 ixy="36.2014E-08"
-                 ixz="${ reflect_y * ( 24.6150E-07 ) }"
-                 iyy="0.0326038"
-                 iyz="${ reflect_y * ( -4.0050E-07 ) }"
-                 izz="0.0201129" />
+        <inertia ixx="0.0040302"
+                 ixy="7.250E-08"
+                 ixz="${ reflect_y * ( 5.2121E-07 ) }"
+                 iyy="0.0067791"
+                 iyz="${ reflect_y * ( -7.9189E-08 ) }"
+                 izz="0.0040286" />
         <!-- ============================================================== -->
       </inertial>

File: pandora_models/pandora_robots_description/urdf/gears/sensors/microphone_sensor.xacro (robot description, xacro)
@@ -2,10 +2,10 @@
 <robot xmlns:xacro="http://ros.org/wiki/xacro" >
   <!-- ==================================================================== -->
-  <xacro:include filename="$(find pandora_sensors_description)/urdf/microphone_sensor.urdf.xacro" />
+  <xacro:include filename="$(find pandora_sensors_description)/urdf/microphone.urdf.xacro" />
   <!-- ==================================================================== -->
 <!-- ###################################################################### -->
   <xacro:macro name="microphone_sensor" >
     <xacro:microphone_caster parent="linear_head_main_link" >
-      <origin xyz="0.00915 -0.02181 0.05251"
+      <origin xyz="-0.02175 -0.0374 0.09643"
               rpy="${zero}" />
     </xacro:microphone_caster>

File: pandora_models/pandora_robots_description/urdf/gears/sensors/sonar_sensor.xacro (robot description, xacro)
@@ -2,10 +2,10 @@
 <robot xmlns:xacro="http://ros.org/wiki/xacro" >
   <!-- ==================================================================== -->
-  <xacro:include filename="$(find pandora_sensors_description)/urdf/sonar_sensor.urdf.xacro" />
+  <xacro:include filename="$(find pandora_sensors_description)/urdf/sonar.urdf.xacro" />
   <!-- ==================================================================== -->
 <!-- ###################################################################### -->
   <!-- ==================================================================== -->
   <xacro:macro name="left_sonar_sensor" >
-    <xacro:sonar_caster name="left"
+    <xacro:sonar_caster prefix_y="left"
                         parent="base_link" >
       <origin xyz="-0.15026 0.06429 0.39925"
@@ -15,5 +15,5 @@
   <!-- ==================================================================== -->
   <xacro:macro name="right_sonar_sensor" >
-    <xacro:sonar_caster name="right"
+    <xacro:sonar_caster prefix_y="right"
                         parent="base_link" >
       <origin xyz="-0.15026 -0.06429 0.39925"

File: pandora_models/pandora_robots_description/urdf/gears/sensors/thermal_sensor.xacro (robot description, xacro)
@@ -2,5 +2,5 @@
 <robot xmlns:xacro="http://ros.org/wiki/xacro" >
   <!-- ==================================================================== -->
-  <xacro:include filename="$(find pandora_sensors_description)/urdf/thermal_sensor.urdf.xacro" />
+  <xacro:include filename="$(find pandora_sensors_description)/urdf/thermal.urdf.xacro" />
   <!-- ==================================================================== -->
 <!-- ###################################################################### -->
@@ -9,6 +9,6 @@
     <xacro:thermal_caster parent="linear_head_main_link"
                           prefix_y="middle" >
-      <origin xyz="0.00915 -0.0373 0.07397"
-              rpy="${zero}" />
+      <origin xyz="0.01575 -0.0614 0.08243"
+              rpy="${-PI_2} 0 0" />
     </xacro:thermal_caster>
   </xacro:macro>
@@ -17,5 +17,5 @@
     <xacro:thermal_caster parent="linear_head_main_link"
                           prefix_y="left" >
-      <origin xyz="-0.00252 0.01037 0.05973"
+      <origin xyz="0.00076 0.01607 0.05800"
               rpy="0 0 ${PI_3}" />
     </xacro:thermal_caster>
@@ -25,5 +25,5 @@
     <xacro:thermal_caster parent="linear_head_main_link"
                           prefix_y="right" >
-      <origin xyz="-0.00252 -0.08511 0.05973"
+      <origin xyz="0.00076 -0.09086 0.05800"
               rpy="0 0 ${-PI_3}" />
     </xacro:thermal_caster>

File: pandora_models/pandora_sensors_description/urdf/co2.urdf.xacro (robot description, xacro)
@@ -2,8 +2,8 @@
 <robot xmlns:xacro="http://ros.org/wiki/xacro" >
 <!-- ###################################################################### -->
-  <xacro:macro name="thermal_caster"
-               params="parent prefix_y *origin" >
+  <xacro:macro name="co2_caster"
+               params="parent *origin" >
     <!-- ################################################################## -->
-    <link name="${prefix_y}_thermal_link" >
+    <link name="co2_link" >
       <inertial>
         <!-- ============================================================== -->
@@ -26,5 +26,5 @@
         <!-- ============================================================== -->
         <geometry>
-          <mesh filename="package://pandora_sensors_description/meshes/thermal_sensor/thermal_small.dae" />
+          <mesh filename="package://pandora_sensors_description/meshes/co2/dynament.dae" />
         </geometry>
         <!-- ============================================================== -->
@@ -32,9 +32,9 @@
       <collision>
         <!-- ============================================================== -->
-        <origin xyz="0.007 0.0 0.0"
+        <origin xyz="0.0075 0.0 0.0"
                 rpy="0 0 0" />
         <!-- ============================================================== -->
         <geometry>
-          <box size="0.025 0.025 0.025" />
+          <box size="0.015 0.022 0.022" />
         </geometry>
         <!-- ============================================================== -->
@@ -42,13 +42,42 @@
     </link>
     <!-- ################################################################## -->
-    <joint name="${prefix_y}_thermal_joint"
+    <link name="co2_frame" >
+      <inertial>
+        <!-- ============================================================== -->
+        <origin xyz="0.0 0.0 0.0" />
+        <!-- ============================================================== -->
+        <mass value="0.0001" />
+        <!-- ============================================================== -->
+        <inertia ixx="0.00000001"
+                 ixy="0"
+                 ixz="0"
+                 iyy="0.00000001"
+                 iyz="0"
+                 izz="0.00000001" />
+        <!-- ============================================================== -->
+      </inertial>
+    </link>
+    <!-- ################################################################## -->
+    <joint name="co2_main_joint"
            type="fixed" >
       <!-- ================================================================ -->
       <parent link="${parent}" />
-      <child link="${prefix_y}_thermal_link" />
+      <child link="co2_link" />
       <!-- ================================================================ -->
       <xacro:insert_block name="origin" />
       <!-- ================================================================ -->
     </joint>
+    <!-- ################################################################## -->
+    <joint name="co2_joint"
+           type="fixed" >
+      <!-- ================================================================ -->
+      <parent link="co2_link" />
+      <child link="co2_frame" />
+      <!-- ================================================================ -->
+      <origin xyz="0.015 0.0 0.0"
+              rpy="0.0 0.0 0.0" />
+      <!-- ================================================================ -->
+    </joint>
+    <!-- ################################################################## -->
   </xacro:macro>
 <!-- ###################################################################### -->

File: pandora_models/pandora_sensors_description/urdf/kinect.urdf.xacro (robot description, xacro)
@@ -69,5 +69,5 @@
         <!-- ============================================================== -->
         <geometry>
-          <mesh filename="package://pandora_sensors_description/meshes/kinect_camera/kinect_base.dae" />
+          <mesh filename="package://pandora_sensors_description/meshes/kinect/base.dae" />
         </geometry>
         <!-- ============================================================== -->
@@ -106,5 +106,5 @@
         <!-- ============================================================== -->
         <geometry>
-          <mesh filename="package://pandora_sensors_description/meshes/kinect_camera/asus_xtion_pro.dae" />
+          <mesh filename="package://pandora_sensors_description/meshes/kinect/asus_xtion_pro.dae" />
         </geometry>
         <!-- ============================================================== -->
@@ -381,4 +381,5 @@
       <!-- ================================================================ -->
     </joint>
+    <!-- ################################################################## -->
   </xacro:macro>
 <!-- ###################################################################### -->

File: pandora_models/pandora_sensors_description/urdf/laser.urdf.xacro (robot description, xacro)
@@ -2,5 +2,5 @@
 <robot xmlns:xacro="http://ros.org/wiki/xacro" >
 <!-- ###################################################################### -->
-  <xacro:macro name="hokuyo_caster"
+  <xacro:macro name="laser_caster"
                params="parent
                        fixed
@@ -32,5 +32,5 @@
         <!-- ============================================================== -->
         <geometry>
-          <mesh filename="package://pandora_sensors_description/meshes/hokuyo_urg_04lx/laser_pitch_servo.dae" />
+          <mesh filename="package://pandora_sensors_description/meshes/laser/pitch_servo_motor.dae" />
         </geometry>
         <!-- ============================================================== -->
@@ -69,5 +69,5 @@
         <!-- ============================================================== -->
         <geometry>
-          <mesh filename="package://pandora_sensors_description/meshes/hokuyo_urg_04lx/hokuyo_urg_04lx.dae" />
+          <mesh filename="package://pandora_sensors_description/meshes/laser/hokuyo_urg_04lx.dae" />
         </geometry>
         <!-- ============================================================== -->
@@ -196,4 +196,5 @@
       <!-- ================================================================ -->
     </joint>
+    <!-- ################################################################## -->
   </xacro:macro>
 <!-- ###################################################################### -->

File: pandora_models/pandora_sensors_description/urdf/microphone.urdf.xacro (robot description, xacro)
@@ -8,5 +8,5 @@
       <inertial>
         <!-- ============================================================== -->
-        <origin xyz="0.005 0.0 0.0" />
+        <origin xyz="0.01177 0.0 0.0" />
         <!-- ============================================================== -->
         <mass value="0.005" />
@@ -26,5 +26,5 @@
         <!-- ============================================================== -->
         <geometry>
-          <mesh filename="package://pandora_sensors_description/meshes/microphone_sensor/microphone_small.dae" />
+          <mesh filename="package://pandora_sensors_description/meshes/microphone/kinect_array.dae" />
         </geometry>
         <!-- ============================================================== -->
@@ -32,9 +32,9 @@
       <collision>
         <!-- ============================================================== -->
-        <origin xyz="0.007 0.0 0.0"
+        <origin xyz="0.0 0.0 0.01"
                 rpy="0 0 0" />
         <!-- ============================================================== -->
         <geometry>
-          <box size="0.025 0.025 0.025" />
+          <box size="0.053 0.055 0.020" />
         </geometry>
         <!-- ============================================================== -->
@@ -42,5 +42,23 @@
     </link>
     <!-- ################################################################## -->
-    <joint name="microphone_joint" type="fixed" >
+    <link name="microphone_frame" >
+      <inertial>
+        <!-- ============================================================== -->
+        <origin xyz="0.0 0.0 0.0" />
+        <!-- ============================================================== -->
+        <mass value="0.0001" />
+        <!-- ============================================================== -->
+        <inertia ixx="0.00000001"
+                 ixy="0"
+                 ixz="0"
+                 iyy="0.00000001"
+                 iyz="0"
+                 izz="0.00000001" />
+        <!-- ============================================================== -->
+      </inertial>
+    </link>
+    <!-- ################################################################## -->
+    <joint name="microphone_main_joint"
+           type="fixed" >
       <!-- ================================================================ -->
       <parent link="${parent}" />
@@ -50,4 +68,16 @@
       <!-- ================================================================ -->
     </joint>
+    <!-- ################################################################## -->
+    <joint name="microphone_joint"
+           type="fixed" >
+      <!-- ================================================================ -->
+      <parent link="microphone_link" />
+      <child link="microphone_frame" />
+      <!-- ================================================================ -->
+      <origin xyz="0.0 0.0 0.0125"
+              rpy="0.0 0.0 0.0" />
+      <!-- ================================================================ -->
+    </joint>
+    <!-- ################################################################## -->
   </xacro:macro>
 <!-- ###################################################################### -->

File: pandora_models/pandora_sensors_description/urdf/sonar.urdf.xacro (robot description, xacro)
@@ -3,7 +3,7 @@
 <!-- ###################################################################### -->
   <xacro:macro name="sonar_caster"
-               params="name parent *origin" >
+               params="parent prefix_y *origin" >
     <!-- ################################################################## -->
-    <link name="${name}_sonar_link" >
+    <link name="${prefix_y}_sonar_link" >
       <inertial>
         <!-- ============================================================== -->
@@ -26,5 +26,5 @@
         <!-- ============================================================== -->
         <geometry>
-          <mesh filename="package://pandora_sensors_description/meshes/sonar_sensor/max_sonar_ez4.dae" />
+          <mesh filename="package://pandora_sensors_description/meshes/sonar/max_ez4.dae" />
         </geometry>
         <!-- ============================================================== -->
@@ -32,9 +32,9 @@
       <collision>
         <!-- ============================================================== -->
-        <origin xyz="0.007 0.0 0.0"
+        <origin xyz="0.0075 0.0 0.0"
                 rpy="0 0 0" />
         <!-- ============================================================== -->
         <geometry>
-          <box size="0.025 0.05 0.025" />
+          <box size="0.015 0.044 0.022" />
         </geometry>
         <!-- ============================================================== -->
@@ -42,13 +42,42 @@
     </link>
     <!-- ################################################################## -->
-    <joint name="${name}_sonar_joint"
+    <link name="${prefix_y}_sonar_frame" >
+      <inertial>
+        <!-- ============================================================== -->
+        <origin xyz="0.0 0.0 0.0" />
+        <!-- ============================================================== -->
+        <mass value="0.0001" />
+        <!-- ============================================================== -->
+        <inertia ixx="0.00000001"
+                 ixy="0"
+                 ixz="0"
+                 iyy="0.00000001"
+                 iyz="0"
+                 izz="0.00000001" />
+        <!-- ============================================================== -->
+      </inertial>
+    </link>
+    <!-- ################################################################## -->
+    <joint name="${prefix_y}_sonar_main_joint"
            type="fixed" >
       <!-- ================================================================ -->
       <parent link="${parent}" />
-      <child link="${name}_sonar_link" />
+      <child link="${prefix_y}_sonar_link" />
       <!-- ================================================================ -->
       <xacro:insert_block name="origin" />
       <!-- ================================================================ -->
     </joint>
+    <!-- ################################################################## -->
+    <joint name="${prefix_y}_sonar_joint"
+           type="fixed" >
+      <!-- ================================================================ -->
+      <parent link="${prefix_y}_sonar_link" />
+      <child link="${prefix_y}_sonar_frame" />
+      <!-- ================================================================ -->
+      <origin xyz="0.015 0.0 0.0"
+              rpy="0.0 0.0 0.0" />
+      <!-- ================================================================ -->
+    </joint>
+    <!-- ################################################################## -->
   </xacro:macro>
 <!-- ###################################################################### -->

File: pandora_models/pandora_sensors_description/urdf/thermal.urdf.xacro (robot description, xacro)
@@ -2,11 +2,11 @@
 <robot xmlns:xacro="http://ros.org/wiki/xacro" >
 <!-- ###################################################################### -->
-  <xacro:macro name="camera_caster"
+  <xacro:macro name="thermal_caster"
                params="parent prefix_y *origin" >
     <!-- ################################################################## -->
-    <link name="${prefix_y}_camera_main_link" >
+    <link name="${prefix_y}_thermal_main_link" >
       <inertial>
         <!-- ============================================================== -->
-        <origin xyz="0.00972 0.0 0.04428" />
+        <origin xyz="0.00126 0.0 0.0" />
         <!-- ============================================================== -->
         <mass value="0.005" />
@@ -26,5 +26,5 @@
         <!-- ============================================================== -->
         <geometry>
-          <mesh filename="package://pandora_sensors_description/meshes/logitech_camera/logitech_camera.dae" />
+          <mesh filename="package://pandora_sensors_description/meshes/thermal/grid_eye.dae" />
         </geometry>
         <!-- ============================================================== -->
@@ -32,9 +32,9 @@
       <collision>
         <!-- ============================================================== -->
-        <origin xyz="0.00557 0.0 0.03624"
+        <origin xyz="0.00225 0.0 0.0"
                 rpy="0 0 0" />
         <!-- ============================================================== -->
         <geometry>
-          <box size="0.049 0.095 0.073" />
+          <box size="0.004 0.020 0.037" />
         </geometry>
         <!-- ============================================================== -->
@@ -42,5 +42,5 @@
     </link>
     <!-- ################################################################## -->
-    <link name="${prefix_y}_camera_frame" >
+    <link name="${prefix_y}_thermal_frame" >
       <inertial>
         <!-- ============================================================== -->
@@ -59,5 +59,5 @@
     </link>
     <!-- ################################################################## -->
-    <link name="${prefix_y}_camera_optical_frame" >
+    <link name="${prefix_y}_thermal_optical_frame" >
       <inertial>
         <!-- ============================================================== -->
@@ -76,9 +76,9 @@
     </link>
     <!-- ################################################################## -->
-    <joint name="${prefix_y}_camera_main_joint"
+    <joint name="${prefix_y}_thermal_main_joint"
            type="fixed" >
       <!-- ================================================================ -->
       <parent link="${parent}" />
-      <child link="${prefix_y}_camera_main_link" />
+      <child link="${prefix_y}_thermal_main_link" />
       <!-- ================================================================ -->
       <xacro:insert_block name="origin" />
@@ -86,20 +86,20 @@
     </joint>
     <!-- ################################################################## -->
-    <joint name="${prefix_y}_camera_joint"
+    <joint name="${prefix_y}_thermal_joint"
            type="fixed" >
       <!-- ================================================================ -->
-      <parent link="${prefix_y}_camera_main_link" />
-      <child link="${prefix_y}_camera_frame" />
+      <parent link="${prefix_y}_thermal_main_link" />
+      <child link="${prefix_y}_thermal_frame" />
       <!-- ================================================================ -->
-      <origin xyz="0.02499 0.0 0.05704"
-              rpy="0.0 -0.2792 0.0" />
+      <origin xyz="0.0045 0.0 0.00125"
+              rpy="0.0 0.0 0.0" />
       <!-- ================================================================ -->
     </joint>
     <!-- ################################################################## -->
-    <joint name="${prefix_y}_camera_optical_joint"
+    <joint name="${prefix_y}_thermal_optical_joint"
            type="fixed" >
       <!-- ================================================================ -->
-      <parent link="${prefix_y}_camera_frame" />
-      <child link="${prefix_y}_camera_optical_frame" />
+      <parent link="${prefix_y}_thermal_frame" />
+      <child link="${prefix_y}_thermal_optical_frame" />
       <!-- ================================================================ -->
       <origin xyz="0.0 0.0 0.0"
