Commit message: Adjust linear's limits and reduce wheels' stiffness.

File: pandora_gazebo/pandora_gazebo_description/urdf/gears/gears_simplified.gazebo.xacro (robot description, xacro)
@@ -21,10 +21,12 @@
   <xacro:include filename="$(find pandora_gazebo_description)/urdf/gears/plugins/ros_control_plugin.gazebo.xacro" />
 <!-- Properties ########################################################### -->
+  <!-- XXX: Get from config -->
   <xacro:property name="robot_namespace" value="" />
-  <xacro:property name="wheel_mu_1" value="0.75" />
-  <xacro:property name="wheel_mu_2" value="0.75" />
-  <xacro:property name="wheel_k_p" value="10000000.0" />
-  <xacro:property name="wheel_k_d" value="1.0" />
+  <xacro:property name="wheel_mu_1" value="0.675" />
+  <xacro:property name="wheel_mu_2" value="0.675" />
+  <xacro:property name="wheel_k_p" value="1000000.0" />
+  <xacro:property name="wheel_k_d" value="0.8" />
   <xacro:property name="wheel_min_depth" value="0.001" />
+  <xacro:property name="wheel_max_contacts" value="1" />
 <!-- Load URDF ############################################################ -->
   <xacro:gears_urdf fixed="false" />

File: pandora_gazebo/pandora_gazebo_description/urdf/gears/sdf_configurations.xacro (robot description, xacro)
@@ -65,9 +65,10 @@
 <!-- Joint Physics ######################################################## -->
   <!-- Wheels ============================================================= -->
-  <xacro:property name="wheel_mu_1" value="0.75" />
-  <xacro:property name="wheel_mu_2" value="0.75" />
-  <xacro:property name="wheel_k_p" value="10000000.0" />
-  <xacro:property name="wheel_k_d" value="1.0" />
+  <xacro:property name="wheel_mu_1" value="0.675" />
+  <xacro:property name="wheel_mu_2" value="0.675" />
+  <xacro:property name="wheel_k_p" value="1000000.0" />
+  <xacro:property name="wheel_k_d" value="0.8" />
   <xacro:property name="wheel_min_depth" value="0.001" />
+  <xacro:property name="wheel_max_contacts" value="1" />
   <!-- ==================================================================== -->
 <!-- Plugin Parameters #################################################### -->

Commit message: Finalize camera sensors.

File: pandora_gazebo/pandora_gazebo_description/urdf/gears/gears_simplified.gazebo.xacro (robot description, xacro)
@@ -8,4 +8,5 @@
   <xacro:include filename="$(find pandora_gazebo_description)/urdf/gears/sensors/laser_sensor.gazebo.xacro" />
   <xacro:include filename="$(find pandora_gazebo_description)/urdf/gears/sensors/kinect_sensor.gazebo.xacro" />
+  <xacro:include filename="$(find pandora_gazebo_description)/urdf/gears/sensors/camera_sensor.gazebo.xacro" />
   <xacro:include filename="$(find pandora_gazebo_description)/urdf/gears/sensors/sonar_sensor.gazebo.xacro" />
   <xacro:include filename="$(find pandora_gazebo_description)/urdf/gears/sensors/thermal_sensor.gazebo.xacro" />
@@ -23,9 +24,9 @@
   <!-- XXX: Get from config -->
   <xacro:property name="robot_namespace" value="" />
-  <xacro:property name="wheel_mu_1" value="0.65" />
-  <xacro:property name="wheel_mu_2" value="0.65" />
-  <xacro:property name="wheel_k_p" value="100000000.0" />
-  <xacro:property name="wheel_k_d" value="0.8" />
-  <xacro:property name="wheel_min_depth" value="0.00001" />
+  <xacro:property name="wheel_mu_1" value="0.45" />
+  <xacro:property name="wheel_mu_2" value="0.45" />
+  <xacro:property name="wheel_k_p" value="10000000.0" />
+  <xacro:property name="wheel_k_d" value="1.0" />
+  <xacro:property name="wheel_min_depth" value="0.0001" />
   <xacro:property name="wheel_max_contacts" value="1" />
 <!-- Load URDF ############################################################ -->
@@ -40,6 +41,8 @@
   <xacro:laser_gazebo_sensor />
   <xacro:kinect_gazebo_sensor />
-  <xacro:sonar_gazebo_sensor name="left" publish_msg="false" />
-  <xacro:sonar_gazebo_sensor name="right" publish_msg="false" />
+  <xacro:camera_gazebo_sensor prefix_y="left" />
+  <xacro:camera_gazebo_sensor prefix_y="right" />
+  <xacro:sonar_gazebo_sensor prefix_y="left" publish_msg="false" />
+  <xacro:sonar_gazebo_sensor prefix_y="right" publish_msg="false" />
   <xacro:co2_gazebo_sensor publish_msg="false" publish_viz="false" />
   <xacro:thermal_gazebo_sensor prefix_y="middle" publish_msg="false" publish_viz="false" />

Commit message: Refactor latest method.

File: pandora_gazebo/pandora_gazebo_description/urdf/gears/gears_simplified.gazebo.xacro (robot description, xacro)
@@ -24,6 +24,6 @@
   <!-- XXX: Get from config -->
   <xacro:property name="robot_namespace" value="" />
-  <xacro:property name="wheel_mu_1" value="0.45" />
-  <xacro:property name="wheel_mu_2" value="0.45" />
+  <xacro:property name="wheel_mu_1" value="0.6" />
+  <xacro:property name="wheel_mu_2" value="0.6" />
   <xacro:property name="wheel_k_p" value="10000000.0" />
   <xacro:property name="wheel_k_d" value="1.0" />

File: pandora_gazebo/pandora_gazebo_description/urdf/gears/sensors/camera_sensor.gazebo.xacro (robot description, xacro)
@@ -28,5 +28,7 @@
           <frameName>${prefix_y}_camera_optical_frame</frameName>
           <!--============================================================= -->
-          <imageTopicName>${prefix_y}_camera/image</imageTopicName>
+          <cameraName>${prefix_y}_camera</cameraName>
+          <!--============================================================= -->
+          <imageTopicName>image</imageTopicName>
           <!--============================================================= -->
         </plugin>

Commit message: Adjust velocity coefficients for new physics.

File: pandora_gazebo/pandora_gazebo_description/urdf/gears/gears_simplified.gazebo.xacro (robot description, xacro)
@@ -25,5 +25,5 @@
   <xacro:property name="robot_namespace" value="" />
   <xacro:property name="wheel_mu_1" value="0.6" />
-  <xacro:property name="wheel_mu_2" value="0.6" />
+  <xacro:property name="wheel_mu_2" value="0.3" />
   <xacro:property name="wheel_k_p" value="10000000.0" />
   <xacro:property name="wheel_k_d" value="1.0" />
