Commit message: Minor adjustment in friction.

File: pandora_gazebo/pandora_gazebo_description/urdf/gears/gears.gazebo.xacro (robot description, xacro)
@@ -80,10 +80,10 @@
     </xacro:if>
     <!-- ================================================================ -->
+    <xacro:if value="${enable_linear_head_yaw_joint_physics}" >
+      <xacro:linear_head_yaw_joint_physics />
+    </xacro:if>
+    <!-- ================================================================ -->
     <xacro:if value="${enable_linear_head_pitch_joint_physics}" >
       <xacro:linear_head_pitch_joint_physics />
-    </xacro:if>
-    <!-- ================================================================ -->
-    <xacro:if value="${enable_linear_head_yaw_joint_physics}" >
-      <xacro:linear_head_yaw_joint_physics />
     </xacro:if>
     <!-- ================================================================ -->

File: pandora_gazebo/pandora_gazebo_description/urdf/gears/gears_simplified.gazebo.xacro (robot description, xacro)
@@ -24,10 +24,10 @@
   <!-- XXX: Get from config -->
   <xacro:property name="robot_namespace" value="" />
-  <xacro:property name="wheel_mu_1" value="0.6" />
-  <xacro:property name="wheel_mu_2" value="0.3" />
+  <xacro:property name="wheel_mu_1" value="0.85" />
+  <xacro:property name="wheel_mu_2" value="0.85" />
   <xacro:property name="wheel_k_p" value="10000000.0" />
   <xacro:property name="wheel_k_d" value="1.0" />
   <xacro:property name="wheel_min_depth" value="0.0001" />
-  <xacro:property name="wheel_max_contacts" value="1" />
+  <xacro:property name="wheel_max_contacts" value="10" />
 <!-- Load URDF ############################################################ -->
   <xacro:gears_urdf fixed="false" />
@@ -57,6 +57,6 @@
   <xacro:wheel_transmission prefix_y="right" prefix_x="rear" />
   <xacro:linear_elevator_transmission />
+  <xacro:linear_head_transmission rotation="yaw" />
   <xacro:linear_head_transmission rotation="pitch" />
-  <xacro:linear_head_transmission rotation="yaw" />
   <xacro:laser_sensor_transmission rotation="roll" />
   <xacro:laser_sensor_transmission rotation="pitch" />

File: pandora_gazebo/pandora_gazebo_description/urdf/gears/sdf_configurations.xacro (robot description, xacro)
@@ -46,6 +46,6 @@
     <xacro:property name="enable_linear_elevator_joint_physics" value="true" />
     <!-- ================================================================== -->
+    <xacro:property name="enable_linear_head_yaw_joint_physics" value="false" />
     <xacro:property name="enable_linear_head_pitch_joint_physics" value="false" />
-    <xacro:property name="enable_linear_head_yaw_joint_physics" value="false" />
     <!-- ================================================================== -->
     <xacro:property name="enable_laser_roll_joint_physics" value="false" />
@@ -70,6 +70,6 @@
 <!-- Joint Physics ######################################################## -->
   <!-- Wheels ============================================================= -->
-  <xacro:property name="wheel_mu_1" value="0.6" />
-  <xacro:property name="wheel_mu_2" value="0.3" />
+  <xacro:property name="wheel_mu_1" value="0.85" />
+  <xacro:property name="wheel_mu_2" value="0.85" />
   <xacro:property name="wheel_k_p" value="10000000.0" />
   <xacro:property name="wheel_k_d" value="1.0" />
