Commit message: Fix roslint errors

File: pandora_gazebo/pandora_gazebo_description/urdf/gears/gears.gazebo.xacro (robot description, xacro)
@@ -153,15 +153,5 @@
           <xacro:if value="${enable_linear_sonar_sensor}" >
             <xacro:if value="${enable_linear_sonar_gazebo_sensor}" >
-              <xacro:if value="$(arg control)" >
-                <xacro:if value="$(arg interface)" >
-                  <xacro:sonar_gazebo_sensor name="linear" publish_msg="false" />
-                </xacro:if>
-                <xacro:unless value="$(arg interface)" >
-                  <xacro:sonar_gazebo_sensor name="linear" publish_msg="true" />
-                </xacro:unless>
-              </xacro:if>
-              <xacro:unless value="$(arg control)" >
-                <xacro:sonar_gazebo_sensor name="linear" publish_msg="true" />
-              </xacro:unless>
+              <xacro:sonar_gazebo_sensor name="linear" />
             </xacro:if>
           </xacro:if>
@@ -169,15 +159,5 @@
           <xacro:if value="${enable_left_sonar_sensor}" >
             <xacro:if value="${enable_left_sonar_gazebo_sensor}" >
-              <xacro:if value="$(arg control)" >
-                <xacro:if value="$(arg interface)" >
-                  <xacro:sonar_gazebo_sensor name="left" publish_msg="false" />
-                </xacro:if>
-                <xacro:unless value="$(arg interface)" >
-                  <xacro:sonar_gazebo_sensor name="left" publish_msg="true" />
-                </xacro:unless>
-              </xacro:if>
-              <xacro:unless value="$(arg control)" >
-                <xacro:sonar_gazebo_sensor name="left" publish_msg="true" />
-              </xacro:unless>
+                  <xacro:sonar_gazebo_sensor name="left" />
             </xacro:if>
           </xacro:if>
@@ -185,15 +165,5 @@
           <xacro:if value="${enable_right_sonar_sensor}" >
             <xacro:if value="${enable_right_sonar_gazebo_sensor}" >
-              <xacro:if value="$(arg control)" >
-                <xacro:if value="$(arg interface)" >
-                  <xacro:sonar_gazebo_sensor name="right" publish_msg="false" />
-                </xacro:if>
-                <xacro:unless value="$(arg interface)" >
-                  <xacro:sonar_gazebo_sensor name="right" publish_msg="true" />
-                </xacro:unless>
-              </xacro:if>
-              <xacro:unless value="$(arg control)" >
-                <xacro:sonar_gazebo_sensor name="right" publish_msg="true" />
-              </xacro:unless>
+                  <xacro:sonar_gazebo_sensor name="right" />
             </xacro:if>
           </xacro:if>
@@ -203,30 +173,5 @@
       <xacro:if value="${enable_co2_sensor}" >
         <xacro:if value="${enable_co2_gazebo_sensor}" >
-          <xacro:if value="$(arg control)" >
-            <xacro:if value="$(arg interface)" >
-              <xacro:if value="$(arg sensors_viz)" >
-                <xacro:co2_gazebo_sensor publish_msg="false" publish_viz="true" />
-              </xacro:if>
-              <xacro:unless value="$(arg sensors_viz)" >
-                <xacro:co2_gazebo_sensor publish_msg="false" publish_viz="false" />
-              </xacro:unless>
-            </xacro:if>
-            <xacro:unless value="$(arg interface)" >
-              <xacro:if value="$(arg sensors_viz)" >
-                <xacro:co2_gazebo_sensor publish_msg="true" publish_viz="true" />
-              </xacro:if>
-              <xacro:unless value="$(arg sensors_viz)" >
-                <xacro:co2_gazebo_sensor publish_msg="true" publish_viz="false" />
-              </xacro:unless>
-            </xacro:unless>
-          </xacro:if>
-          <xacro:unless value="$(arg control)" >
-            <xacro:if value="$(arg sensors_viz)" >
-              <xacro:co2_gazebo_sensor publish_msg="true" publish_viz="true" />
-            </xacro:if>
-            <xacro:unless value="$(arg sensors_viz)" >
-              <xacro:co2_gazebo_sensor publish_msg="true" publish_viz="false" />
-            </xacro:unless>
-          </xacro:unless>
+                <xacro:co2_gazebo_sensor />
         </xacro:if>
       </xacro:if>
@@ -236,30 +181,5 @@
           <xacro:if value="${enable_middle_thermal_sensor}" >
             <xacro:if value="${enable_middle_thermal_gazebo_sensor}" >
-              <xacro:if value="$(arg control)" >
-                <xacro:if value="$(arg interface)" >
-                  <xacro:if value="$(arg sensors_viz)" >
-                    <xacro:thermal_gazebo_sensor prefix_y="middle" publish_msg="false" publish_viz="true" />
-                  </xacro:if>
-                  <xacro:unless value="$(arg sensors_viz)" >
-                    <xacro:thermal_gazebo_sensor prefix_y="middle" publish_msg="false" publish_viz="false" />
-                  </xacro:unless>
-                </xacro:if>
-                <xacro:unless value="$(arg interface)" >
-                  <xacro:if value="$(arg sensors_viz)" >
-                    <xacro:thermal_gazebo_sensor prefix_y="middle" publish_msg="true" publish_viz="true" />
-                  </xacro:if>
-                  <xacro:unless value="$(arg sensors_viz)" >
-                    <xacro:thermal_gazebo_sensor prefix_y="middle" publish_msg="true" publish_viz="false" />
-                  </xacro:unless>
-                </xacro:unless>
-              </xacro:if>
-              <xacro:unless value="$(arg control)" >
-                <xacro:if value="$(arg sensors_viz)" >
-                  <xacro:thermal_gazebo_sensor prefix_y="middle" publish_msg="true" publish_viz="true" />
-                </xacro:if>
-                <xacro:unless value="$(arg sensors_viz)" >
-                  <xacro:thermal_gazebo_sensor prefix_y="middle" publish_msg="true" publish_viz="false" />
-                </xacro:unless>
-              </xacro:unless>
+                    <xacro:thermal_gazebo_sensor prefix_y="middle" />
             </xacro:if>
           </xacro:if>
@@ -267,30 +187,5 @@
           <xacro:if value="${enable_left_thermal_sensor}" >
             <xacro:if value="${enable_left_thermal_gazebo_sensor}" >
-              <xacro:if value="$(arg control)" >
-                <xacro:if value="$(arg interface)" >
-                  <xacro:if value="$(arg sensors_viz)" >
-                    <xacro:thermal_gazebo_sensor prefix_y="left" publish_msg="false" publish_viz="true" />
-                  </xacro:if>
-                  <xacro:unless value="$(arg sensors_viz)" >
-                    <xacro:thermal_gazebo_sensor prefix_y="left" publish_msg="false" publish_viz="false" />
-                  </xacro:unless>
-                </xacro:if>
-                <xacro:unless value="$(arg interface)" >
-                  <xacro:if value="$(arg sensors_viz)" >
-                    <xacro:thermal_gazebo_sensor prefix_y="left" publish_msg="true" publish_viz="true" />
-                  </xacro:if>
-                  <xacro:unless value="$(arg sensors_viz)" >
-                    <xacro:thermal_gazebo_sensor prefix_y="left" publish_msg="true" publish_viz="false" />
-                  </xacro:unless>
-                </xacro:unless>
-              </xacro:if>
-              <xacro:unless value="$(arg control)" >
-                <xacro:if value="$(arg sensors_viz)" >
-                  <xacro:thermal_gazebo_sensor prefix_y="left" publish_msg="true" publish_viz="true" />
-                </xacro:if>
-                <xacro:unless value="$(arg sensors_viz)" >
-                  <xacro:thermal_gazebo_sensor prefix_y="left" publish_msg="true" publish_viz="false" />
-                </xacro:unless>
-              </xacro:unless>
+                    <xacro:thermal_gazebo_sensor prefix_y="left" />
             </xacro:if>
           </xacro:if>
@@ -298,30 +193,5 @@
           <xacro:if value="${enable_right_thermal_sensor}" >
             <xacro:if value="${enable_right_thermal_gazebo_sensor}" >
-              <xacro:if value="$(arg control)" >
-                <xacro:if value="$(arg interface)" >
-                  <xacro:if value="$(arg sensors_viz)" >
-                    <xacro:thermal_gazebo_sensor prefix_y="right" publish_msg="false" publish_viz="true" />
-                  </xacro:if>
-                  <xacro:unless value="$(arg sensors_viz)" >
-                    <xacro:thermal_gazebo_sensor prefix_y="right" publish_msg="false" publish_viz="false" />
-                  </xacro:unless>
-                </xacro:if>
-                <xacro:unless value="$(arg interface)" >
-                  <xacro:if value="$(arg sensors_viz)" >
-                    <xacro:thermal_gazebo_sensor prefix_y="right" publish_msg="true" publish_viz="true" />
-                  </xacro:if>
-                  <xacro:unless value="$(arg sensors_viz)" >
-                    <xacro:thermal_gazebo_sensor prefix_y="right" publish_msg="true" publish_viz="false" />
-                  </xacro:unless>
-                </xacro:unless>
-              </xacro:if>
-              <xacro:unless value="$(arg control)" >
-                <xacro:if value="$(arg sensors_viz)" >
-                  <xacro:thermal_gazebo_sensor prefix_y="right" publish_msg="true" publish_viz="true" />
-                </xacro:if>
-                <xacro:unless value="$(arg sensors_viz)" >
-                  <xacro:thermal_gazebo_sensor prefix_y="right" publish_msg="true" publish_viz="false" />
-                </xacro:unless>
-              </xacro:unless>
+                    <xacro:thermal_gazebo_sensor prefix_y="right" />
             </xacro:if>
           </xacro:if>
@@ -331,30 +201,5 @@
       <xacro:if value="${enable_microphone_sensor}" >
         <xacro:if value="${enable_microphone_gazebo_sensor}" >
-          <xacro:if value="$(arg control)" >
-            <xacro:if value="$(arg interface)" >
-              <xacro:if value="$(arg sensors_viz)" >
-                <xacro:microphone_gazebo_sensor publish_msg="false" publish_viz="true" />
-              </xacro:if>
-              <xacro:unless value="$(arg sensors_viz)" >
-                <xacro:microphone_gazebo_sensor publish_msg="false" publish_viz="false" />
-              </xacro:unless>
-            </xacro:if>
-            <xacro:unless value="$(arg interface)" >
-              <xacro:if value="$(arg sensors_viz)" >
-                <xacro:microphone_gazebo_sensor publish_msg="true" publish_viz="true" />
-              </xacro:if>
-              <xacro:unless value="$(arg sensors_viz)" >
-                <xacro:microphone_gazebo_sensor publish_msg="true" publish_viz="false" />
-              </xacro:unless>
-            </xacro:unless>
-          </xacro:if>
-          <xacro:unless value="$(arg control)" >
-            <xacro:if value="$(arg sensors_viz)" >
-              <xacro:microphone_gazebo_sensor publish_msg="true" publish_viz="true" />
-            </xacro:if>
-            <xacro:unless value="$(arg sensors_viz)" >
-              <xacro:microphone_gazebo_sensor publish_msg="true" publish_viz="false" />
-            </xacro:unless>
-          </xacro:unless>
+                <xacro:microphone_gazebo_sensor />
         </xacro:if>
       </xacro:if>
@@ -431,5 +276,5 @@
     <xacro:if value="$(arg interface)" >
       <xacro:gazebo_ros_control_plugin namespace="/"
-                                       hardware_interface="pandora_gazebo_interface/GazeboInterface" />
+                                       hardware_interface="pandora_gazebo_interface/GearsGazeboInterface" />
     </xacro:if>
     <xacro:unless value="$(arg interface)" >

File: pandora_gazebo/pandora_gazebo_description/urdf/gears/gears_simplified.gazebo.xacro (robot description, xacro)
@@ -45,12 +45,12 @@
   <xacro:camera_gazebo_sensor prefix_y="left" />
   <xacro:camera_gazebo_sensor prefix_y="right" />
-  <xacro:sonar_gazebo_sensor name="linear" publish_msg="false" />
-  <xacro:sonar_gazebo_sensor name="left" publish_msg="false" />
-  <xacro:sonar_gazebo_sensor name="right" publish_msg="false" />
-  <xacro:co2_gazebo_sensor publish_msg="false" publish_viz="false" />
-  <xacro:thermal_gazebo_sensor prefix_y="middle" publish_msg="false" publish_viz="false" />
-  <xacro:thermal_gazebo_sensor prefix_y="left" publish_msg="false" publish_viz="false" />
-  <xacro:thermal_gazebo_sensor prefix_y="right" publish_msg="false" publish_viz="false" />
-  <xacro:microphone_gazebo_sensor publish_msg="false" publish_viz="false" />
+  <xacro:sonar_gazebo_sensor name="linear" />
+  <xacro:sonar_gazebo_sensor name="left" />
+  <xacro:sonar_gazebo_sensor name="right" />
+  <xacro:co2_gazebo_sensor />
+  <xacro:thermal_gazebo_sensor prefix_y="middle" />
+  <xacro:thermal_gazebo_sensor prefix_y="left" />
+  <xacro:thermal_gazebo_sensor prefix_y="right" />
+  <xacro:microphone_gazebo_sensor />
 <!-- Load Transmissions ################################################### -->
   <xacro:wheel_transmission prefix_y="left" prefix_x="front" />
@@ -69,5 +69,5 @@
   <xacro:pandora_p3d_plugin />
   <xacro:gazebo_ros_control_plugin namespace="/"
-                                   hardware_interface="pandora_gazebo_interface/GazeboInterface" />
+                                   hardware_interface="pandora_gazebo_interface/GearsGazeboInterface" />
 <!--  <xacro:pandora_wheel_physics_plugin /> -->
 <!--  <xacro:pandora_fdir_plugin /> -->

File: pandora_gazebo/pandora_gazebo_description/urdf/gears/sensors/co2_sensor.gazebo.xacro (robot description, xacro)
@@ -2,6 +2,5 @@
 <robot xmlns:xacro="http://ros.org/wiki/xacro" >
 <!-- ###################################################################### -->
-  <xacro:macro name="co2_gazebo_sensor"
-               params="publish_msg publish_viz" >
+  <xacro:macro name="co2_gazebo_sensor" >
     <gazebo reference="co2_frame" >
       <sensor name="co2"
@@ -12,12 +11,6 @@
           <!--============================================================= -->
           <image>
-            <xacro:if value="${publish_viz}" >
-              <width>640</width>
-              <height>480</height>
-            </xacro:if>
-            <xacro:unless value="${publish_viz}" >
-              <width>8</width>
-              <height>8</height>
-            </xacro:unless>
+            <width>8</width>
+            <height>8</height>
           </image>
           <!--============================================================= -->
@@ -30,12 +23,9 @@
         <plugin name="co2ros"
                 filename="libpandora_gazebo_plugins_pandora_co2_plugin.so" >
+          <robotNamespace>gazebo_sensors</robotNamespace>
           <!--============================================================= -->
           <frameName>co2_frame</frameName>
           <!--============================================================= -->
-          <topicName>sensors/co2</topicName>
-          <!--============================================================= -->
-          <publishMsg>${publish_msg}</publishMsg>
-          <!--============================================================= -->
-          <publishViz>${publish_viz}</publishViz>
+          <topicName>co2</topicName>
           <!--============================================================= -->
         </plugin>

File: pandora_gazebo/pandora_gazebo_description/urdf/gears/sensors/microphone_sensor.gazebo.xacro (robot description, xacro)
@@ -2,6 +2,5 @@
 <robot xmlns:xacro="http://ros.org/wiki/xacro" >
 <!-- ###################################################################### -->
-  <xacro:macro name="microphone_gazebo_sensor"
-               params="publish_msg publish_viz" >
+  <xacro:macro name="microphone_gazebo_sensor" >
     <gazebo reference="microphone_frame" >
       <sensor name="microphone"
@@ -12,12 +11,6 @@
           <!--============================================================= -->
           <image>
-            <xacro:if value="${publish_viz}" >
-              <width>640</width>
-              <height>480</height>
-            </xacro:if>
-            <xacro:unless value="${publish_viz}" >
-              <width>8</width>
-              <height>8</height>
-            </xacro:unless>
+            <width>8</width>
+            <height>8</height>
           </image>
           <!--============================================================= -->
@@ -30,12 +23,9 @@
         <plugin name="microphone2ros"
                 filename="libpandora_gazebo_plugins_pandora_microphone_plugin.so" >
+          <robotNamespace>gazebo_sensors</robotNamespace>
           <!--============================================================= -->
           <frameName>microphone_frame</frameName>
           <!--============================================================= -->
-          <topicName>sensors/sound</topicName>
-          <!--============================================================= -->
-          <publishMsg>${publish_msg}</publishMsg>
-          <!--============================================================= -->
-          <publishViz>${publish_viz}</publishViz>
+          <topicName>sound</topicName>
           <!--============================================================= -->
         </plugin>

File: pandora_gazebo/pandora_gazebo_description/urdf/gears/sensors/sonar_sensor.gazebo.xacro (robot description, xacro)
@@ -3,5 +3,5 @@
 <!-- ###################################################################### -->
   <xacro:macro name="sonar_gazebo_sensor"
-               params="name publish_msg" >
+               params="name" >
     <gazebo reference="${name}_sonar_frame" >
       <sensor name="${name}_sonar"
@@ -36,14 +36,11 @@
         <plugin name="sonar2ros"
                 filename="libpandora_gazebo_plugins_pandora_sonar_plugin.so" >
-          <!--============================================================= -->
-          <robotNamespace></robotNamespace>
+          <robotNamespace>gazebo_sensors</robotNamespace>
           <!--============================================================= -->
           <frameName>${name}_sonar_frame</frameName>
           <!--============================================================= -->
-          <topicName>/sensors/sonar</topicName> <!-- FIXME -->
+          <topicName>range</topicName>
           <!--============================================================= -->
           <gaussianNoise>0.0</gaussianNoise>
-          <!--============================================================= -->
-          <publishMsg>${publish_msg}</publishMsg>
           <!--============================================================= -->
         </plugin>

File: pandora_gazebo/pandora_gazebo_description/urdf/gears/sensors/thermal_sensor.gazebo.xacro (robot description, xacro)
@@ -3,5 +3,5 @@
 <!-- ###################################################################### -->
   <xacro:macro name="thermal_gazebo_sensor"
-               params="prefix_y publish_msg publish_viz" >
+               params="prefix_y" >
     <gazebo reference="${prefix_y}_thermal_frame" >
       <sensor name="${prefix_y}_thermal"
@@ -12,12 +12,6 @@
           <!--============================================================= -->
           <image>
-            <xacro:if value="${publish_viz}" >
-              <width>640</width>
-              <height>480</height>
-            </xacro:if>
-            <xacro:unless value="${publish_viz}" >
-              <width>8</width>
-              <height>8</height>
-            </xacro:unless>
+            <width>8</width>
+            <height>8</height>
           </image>
           <!--============================================================= -->
@@ -30,12 +24,9 @@
         <plugin name="thermal2ros"
                 filename="libpandora_gazebo_plugins_pandora_thermal_plugin.so" >
+          <robotNamespace>gazebo_sensors</robotNamespace>
           <!--============================================================= -->
           <frameName>${prefix_y}_thermal_optical_frame</frameName>
           <!--============================================================= -->
-          <topicName>sensors/thermal</topicName>
-          <!--============================================================= -->
-          <publishMsg>${publish_msg}</publishMsg>
-          <!--============================================================= -->
-          <publishViz>${publish_viz}</publishViz>
+          <topicName>thermal</topicName>
           <!--============================================================= -->
         </plugin>

File: pandora_gazebo/pandora_gazebo_description/urdf/woody/sdf_configurations.xacro (robot description, xacro)
@@ -9,5 +9,19 @@
   <xacro:property name="static_robot" value="false" />
   <!-- ==================================================================== -->
-  <!-- Sensors ============================================================ -->
+  <!-- Model Sensors ====================================================== -->
+   <!-- FIXME: Remove all model properties (should be set in URDF) -->
+  <xacro:property name="enable_sensors" value="true" />
+    <xacro:property name="enable_laser_sensor" value="true" />
+    <xacro:property name="enable_kinect_sensor" value="true" />
+    <xacro:property name="enable_camera_sensors" value="true" />
+      <xacro:property name="enable_left_camera_sensor" value="true" />
+      <xacro:property name="enable_right_camera_sensor" value="true" />
+    <xacro:property name="enable_sonar_sensors" value="true" />
+      <xacro:property name="enable_left_sonar_sensor" value="true" />
+      <xacro:property name="enable_right_sonar_sensor" value="true" />
+    <xacro:property name="enable_thermal_sensor" value="false" />
+    <xacro:property name="enable_co2_sensor" value="true" />
+    <xacro:property name="enable_microphone_sensor" value="false" />
+  <!-- Gazebo Sensors ===================================================== -->
   <xacro:property name="enable_gazebo_sensors" value="true" />
     <!-- ================================================================== -->
@@ -24,5 +38,5 @@
       <xacro:property name="enable_right_sonar_gazebo_sensor" value="true" />
     <!-- ================================================================== -->
-    <xacro:property name="enable_thermal_gazebo_sensor" value="true" />
+    <xacro:property name="enable_thermal_gazebo_sensor" value="false" />
     <!-- ================================================================== -->
     <xacro:property name="enable_co2_gazebo_sensor" value="true" />
