Commit message: Fix roslint errors

File: pandora_gazebo/pandora_gazebo_description/urdf/woody/sensors/sonar_sensor.gazebo.xacro (robot description, xacro)
@@ -3,5 +3,5 @@
 <!-- ###################################################################### -->
   <xacro:macro name="sonar_gazebo_sensor"
-               params="name publish_msg" >
+               params="name" >
     <gazebo reference="${name}_sonar_frame" >
       <sensor name="${name}_sonar"
@@ -37,13 +37,11 @@
                 filename="libpandora_gazebo_plugins_pandora_sonar_plugin.so" >
           <!--============================================================= -->
-          <robotNamespace></robotNamespace>
+          <robotNamespace>gazebo_sensors</robotNamespace>
           <!--============================================================= -->
           <frameName>${name}_sonar_frame</frameName>
           <!--============================================================= -->
-          <topicName>/sensors/sonar</topicName> <!-- FIXME -->
+          <topicName>range</topicName>
           <!--============================================================= -->
           <gaussianNoise>0.0</gaussianNoise>
-          <!--============================================================= -->
-          <publishMsg>${publish_msg}</publishMsg>
           <!--============================================================= -->
         </plugin>

File: pandora_gazebo/pandora_gazebo_description/urdf/woody/woody.gazebo.xacro (robot description, xacro)
@@ -135,15 +135,5 @@
           <xacro:if value="${enable_left_sonar_sensor}" >
             <xacro:if value="${enable_left_sonar_gazebo_sensor}" >
-              <xacro:if value="$(arg control)" >
-                <xacro:if value="$(arg interface)" >
-                  <xacro:sonar_gazebo_sensor name="left" publish_msg="false" />
-                </xacro:if>
-                <xacro:unless value="$(arg interface)" >
-                  <xacro:sonar_gazebo_sensor name="left" publish_msg="true" />
-                </xacro:unless>
-              </xacro:if>
-              <xacro:unless value="$(arg control)" >
-                <xacro:sonar_gazebo_sensor name="left" publish_msg="true" />
-              </xacro:unless>
+              <xacro:sonar_gazebo_sensor name="left" />
             </xacro:if>
           </xacro:if>
@@ -151,15 +141,5 @@
           <xacro:if value="${enable_right_sonar_sensor}" >
             <xacro:if value="${enable_right_sonar_gazebo_sensor}" >
-              <xacro:if value="$(arg control)" >
-                <xacro:if value="$(arg interface)" >
-                  <xacro:sonar_gazebo_sensor name="right" publish_msg="false" />
-                </xacro:if>
-                <xacro:unless value="$(arg interface)" >
-                  <xacro:sonar_gazebo_sensor name="right" publish_msg="true" />
-                </xacro:unless>
-              </xacro:if>
-              <xacro:unless value="$(arg control)" >
-                <xacro:sonar_gazebo_sensor name="right" publish_msg="true" />
-              </xacro:unless>
+              <xacro:sonar_gazebo_sensor name="right" />
             </xacro:if>
           </xacro:if>
@@ -169,61 +149,11 @@
       <xacro:if value="${enable_co2_sensor}" >
         <xacro:if value="${enable_co2_gazebo_sensor}" >
-          <xacro:if value="$(arg control)" >
-            <xacro:if value="$(arg interface)" >
-              <xacro:if value="$(arg sensors_viz)" >
-                <xacro:co2_gazebo_sensor publish_msg="false" publish_viz="true" />
-              </xacro:if>
-              <xacro:unless value="$(arg sensors_viz)" >
-                <xacro:co2_gazebo_sensor publish_msg="false" publish_viz="false" />
-              </xacro:unless>
-            </xacro:if>
-            <xacro:unless value="$(arg interface)" >
-              <xacro:if value="$(arg sensors_viz)" >
-                <xacro:co2_gazebo_sensor publish_msg="true" publish_viz="true" />
-              </xacro:if>
-              <xacro:unless value="$(arg sensors_viz)" >
-                <xacro:co2_gazebo_sensor publish_msg="true" publish_viz="false" />
-              </xacro:unless>
-            </xacro:unless>
-          </xacro:if>
-          <xacro:unless value="$(arg control)" >
-            <xacro:if value="$(arg sensors_viz)" >
-              <xacro:co2_gazebo_sensor publish_msg="true" publish_viz="true" />
-            </xacro:if>
-            <xacro:unless value="$(arg sensors_viz)" >
-              <xacro:co2_gazebo_sensor publish_msg="true" publish_viz="false" />
-            </xacro:unless>
-          </xacro:unless>
-        </xacro:if>
-      </xacro:if>
-      <xacro:if value="${enable_thermal_sensors}" >
+          <xacro:co2_gazebo_sensor />
+        </xacro:if>
+      </xacro:if>
+      <xacro:if value="${enable_thermal_sensor}" >
         <xacro:if value="${enable_thermal_gazebo_sensor}" >
           <xacro:if value="${enable_thermal_gazebo_sensor}" >
-            <xacro:if value="$(arg control)" >
-              <xacro:if value="$(arg interface)" >
-                <xacro:if value="$(arg sensors_viz)" >
-                  <xacro:thermal_gazebo_sensor prefix_y="middle" publish_msg="false" publish_viz="true" />
-                </xacro:if>
-                <xacro:unless value="$(arg sensors_viz)" >
-                  <xacro:thermal_gazebo_sensor prefix_y="middle" publish_msg="false" publish_viz="false" />
-                </xacro:unless>
-              </xacro:if>
-              <xacro:unless value="$(arg interface)" >
-                <xacro:if value="$(arg sensors_viz)" >
-                  <xacro:thermal_gazebo_sensor prefix_y="middle" publish_msg="true" publish_viz="true" />
-                </xacro:if>
-                <xacro:unless value="$(arg sensors_viz)" >
-                  <xacro:thermal_gazebo_sensor prefix_y="middle" publish_msg="true" publish_viz="false" />
-                </xacro:unless>
-              </xacro:unless>
-            </xacro:if>
-            <xacro:unless value="$(arg control)" >
-              <xacro:if value="$(arg sensors_viz)" >
-                <xacro:thermal_gazebo_sensor prefix_y="middle" publish_msg="true" publish_viz="true" />
-              </xacro:if>
-              <xacro:unless value="$(arg sensors_viz)" >
-                <xacro:thermal_gazebo_sensor prefix_y="middle" publish_msg="true" publish_viz="false" />
-              </xacro:unless>
-            </xacro:unless>
+            <xacro:thermal_gazebo_sensor prefix_y="middle" />
           </xacro:if>
         </xacro:if>
@@ -231,30 +161,5 @@
       <xacro:if value="${enable_microphone_sensor}" >
         <xacro:if value="${enable_microphone_gazebo_sensor}" >
-          <xacro:if value="$(arg control)" >
-            <xacro:if value="$(arg interface)" >
-              <xacro:if value="$(arg sensors_viz)" >
-                <xacro:microphone_gazebo_sensor publish_msg="false" publish_viz="true" />
-              </xacro:if>
-              <xacro:unless value="$(arg sensors_viz)" >
-                <xacro:microphone_gazebo_sensor publish_msg="false" publish_viz="false" />
-              </xacro:unless>
-            </xacro:if>
-            <xacro:unless value="$(arg interface)" >
-              <xacro:if value="$(arg sensors_viz)" >
-                <xacro:microphone_gazebo_sensor publish_msg="true" publish_viz="true" />
-              </xacro:if>
-              <xacro:unless value="$(arg sensors_viz)" >
-                <xacro:microphone_gazebo_sensor publish_msg="true" publish_viz="false" />
-              </xacro:unless>
-            </xacro:unless>
-          </xacro:if>
-          <xacro:unless value="$(arg control)" >
-            <xacro:if value="$(arg sensors_viz)" >
-              <xacro:microphone_gazebo_sensor publish_msg="true" publish_viz="true" />
-            </xacro:if>
-            <xacro:unless value="$(arg sensors_viz)" >
-              <xacro:microphone_gazebo_sensor publish_msg="true" publish_viz="false" />
-            </xacro:unless>
-          </xacro:unless>
+          <xacro:microphone_gazebo_sensor />
         </xacro:if>
       </xacro:if>
@@ -328,5 +233,5 @@
     <xacro:if value="$(arg interface)" >
       <xacro:gazebo_ros_control_plugin namespace="/"
-                                       hardware_interface="pandora_gazebo_interface/GazeboInterface" />
+                                       hardware_interface="pandora_gazebo_interface/WoodyGazeboInterface" />
     </xacro:if>
     <xacro:unless value="$(arg interface)" >

File: pandora_gazebo/pandora_gazebo_description/urdf/woody/woody_simplified.gazebo.xacro (robot description, xacro)
@@ -43,10 +43,8 @@
 <!--  <xacro:camera_gazebo_sensor prefix_y="left" />-->
 <!--  <xacro:camera_gazebo_sensor prefix_y="right" />-->
-  <xacro:sonar_gazebo_sensor name="left" publish_msg="false" />
-  <xacro:sonar_gazebo_sensor name="right" publish_msg="false" />
-<!--  TODO: <xacro:flir_gazebo_sensor publish_msg="false" publish_viz="false" />-->
-<!--  <xacro:co2_gazebo_sensor publish_msg="false" publish_viz="false" />-->
-<!--  <xacro:thermal_gazebo_sensor prefix_y="middle" publish_msg="false" publish_viz="false" />-->
-<!--  <xacro:microphone_gazebo_sensor publish_msg="false" publish_viz="false" />-->
+  <xacro:sonar_gazebo_sensor name="left" />
+  <xacro:sonar_gazebo_sensor name="right" />
+<!--  <xacro:flir_gazebo_sensor />--> <!-- TODO -->
+  <xacro:co2_gazebo_sensor />
 <!-- Load Transmissions ################################################### -->
   <xacro:wheel_transmission prefix_y="left" prefix_x="front" />
@@ -59,16 +57,10 @@
   <xacro:kinect_sensor_transmission rotation="pitch" />
 <!-- Load Plugins ######################################################### -->
-  <xacro:ros_skid_steer_drive_plugin />
-  <xacro:property name="wheel_joint_max_torque" value="50" />
-  <xacro:pandora_differential_plugin publish_joint_states="true" />
-<!-- <xacro:pandora_differential_plugin publish_joint_states="false" /> -->
-  <xacro:pandora_imu_stabilizer_plugin />
-<!-- <xacro:pandora_p3d_plugin /> -->
+  <xacro:pandora_differential_plugin publish_joint_states="false" />
+  <xacro:pandora_p3d_plugin />
   <xacro:gazebo_ros_control_plugin namespace="/"
-                                   hardware_interface="gazebo_ros_control/DefaultRobotHWSim" />
-<!-- <xacro:gazebo_ros_control_plugin namespace="/"
-                                      hardware_interface="pandora_gazebo_interface/GazeboInterface" /> -->
-<!-- <xacro:pandora_wheel_physics_plugin/> -->
-<!-- <xacro:pandora_fdir_plugin />-->
+                                   hardware_interface="pandora_gazebo_interface/WoodyGazeboInterface" />
+<!--  <xacro:pandora_wheel_physics_plugin/> -->
+<!--  <xacro:pandora_fdir_plugin />-->
 <!-- ###################################################################### -->
 </robot>
