Commit message: Enable imu_stabilizer_plugin [ci skip]

File: pandora_gazebo/pandora_gazebo_description/urdf/woody/woody_simplified.gazebo.xacro (robot description, xacro)
@@ -18,4 +18,5 @@
   <xacro:include filename="$(find pandora_gazebo_description)/urdf/woody/plugins/pandora_p3d_plugin.gazebo.xacro" />
   <xacro:include filename="$(find pandora_gazebo_description)/urdf/woody/plugins/ros_control_plugin.gazebo.xacro" />
+  <xacro:include filename="$(find pandora_gazebo_description)/urdf/woody/plugins/pandora_imu_stabilizer_plugin.gazebo.xacro" />
   <xacro:include filename="$(find pandora_gazebo_description)/urdf/woody/plugins/ros_skid_steer_drive_plugin.gazebo.xacro" />
   <xacro:include filename="$(find pandora_gazebo_description)/urdf/gears/plugins/pandora_wheel_physics_plugin.gazebo.xacro" />
@@ -24,6 +25,6 @@
   <!-- XXX: Get from config -->
   <xacro:property name="robot_namespace" value="" />
-  <xacro:property name="wheel_mu_1" value="0.35" />
-  <xacro:property name="wheel_mu_2" value="0.35" />
+  <xacro:property name="wheel_mu_1" value="0.90" />
+  <xacro:property name="wheel_mu_2" value="0.90" />
   <xacro:property name="wheel_k_p" value="10000000.0" />
   <xacro:property name="wheel_k_d" value="1.0" />
@@ -31,6 +32,5 @@
   <xacro:property name="wheel_max_contacts" value="5" />
 <!-- Load URDF ############################################################ -->
-  <!-- <xacro:woody_urdf fixed="false" /> -->
-  <xacro:woody_urdf fixed="true" />
+  <xacro:woody_urdf fixed="false" />
 <!-- Load Physics ######################################################### -->
   <xacro:wheel_link_physics prefix_y="left" prefix_x="front" />
@@ -41,25 +41,21 @@
   <xacro:laser_gazebo_sensor />
   <xacro:kinect_gazebo_sensor />
-  <!--
-  <xacro:camera_gazebo_sensor prefix_y="left" />
-  <xacro:camera_gazebo_sensor prefix_y="right" />
-  TODO: <xacro:flir_gazebo_sensor publish_msg="false" publish_viz="false" />
+<!--  <xacro:camera_gazebo_sensor prefix_y="left" />-->
+<!--  <xacro:camera_gazebo_sensor prefix_y="right" />-->
   <xacro:sonar_gazebo_sensor name="left" publish_msg="false" />
   <xacro:sonar_gazebo_sensor name="right" publish_msg="false" />
-  <xacro:co2_gazebo_sensor publish_msg="false" publish_viz="false" />
-  FIXME: <xacro:thermal_gazebo_sensor prefix_y="middle" publish_msg="false" publish_viz="false" />
-  <xacro:microphone_gazebo_sensor publish_msg="false" publish_viz="false" />
-  -->
+<!--  TODO: <xacro:flir_gazebo_sensor publish_msg="false" publish_viz="false" />-->
+<!--  <xacro:co2_gazebo_sensor publish_msg="false" publish_viz="false" />-->
+<!--  <xacro:thermal_gazebo_sensor prefix_y="middle" publish_msg="false" publish_viz="false" />-->
+<!--  <xacro:microphone_gazebo_sensor publish_msg="false" publish_viz="false" />-->
 <!-- Load Transmissions ################################################### -->
-<!--  <xacro:wheel_transmission prefix_y="left" prefix_x="front" />-->
-<!--  <xacro:wheel_transmission prefix_y="left" prefix_x="rear" />-->
-<!--  <xacro:wheel_transmission prefix_y="right" prefix_x="front" />-->
-<!--  <xacro:wheel_transmission prefix_y="right" prefix_x="rear" />-->
-<!--  -->
-<!--  <xacro:laser_sensor_transmission rotation="roll" />-->
-<!--  <xacro:laser_sensor_transmission rotation="pitch" />-->
-<!--  -->
-<!--  <xacro:kinect_sensor_transmission rotation="pitch" />-->
-<!--  <xacro:kinect_sensor_transmission rotation="yaw" />-->
+  <xacro:wheel_transmission prefix_y="left" prefix_x="front" />
+  <xacro:wheel_transmission prefix_y="left" prefix_x="rear" />
+  <xacro:wheel_transmission prefix_y="right" prefix_x="front" />
+  <xacro:wheel_transmission prefix_y="right" prefix_x="rear" />
+  <xacro:laser_sensor_transmission rotation="roll" />
+  <xacro:laser_sensor_transmission rotation="pitch" />
+  <xacro:kinect_sensor_transmission rotation="yaw" />
+  <xacro:kinect_sensor_transmission rotation="pitch" />
 <!-- Load Plugins ######################################################### -->
   <xacro:ros_skid_steer_drive_plugin />
@@ -67,7 +63,8 @@
   <xacro:pandora_differential_plugin publish_joint_states="true" />
 <!-- <xacro:pandora_differential_plugin publish_joint_states="false" /> -->
+  <xacro:pandora_imu_stabilizer_plugin />
 <!-- <xacro:pandora_p3d_plugin /> -->
-<!--  <xacro:gazebo_ros_control_plugin namespace="/"-->
-<!--                                   hardware_interface="gazebo_ros_control/DefaultRobotHWSim" />-->
+  <xacro:gazebo_ros_control_plugin namespace="/"
+                                   hardware_interface="gazebo_ros_control/DefaultRobotHWSim" />
 <!-- <xacro:gazebo_ros_control_plugin namespace="/"
                                       hardware_interface="pandora_gazebo_interface/GazeboInterface" /> -->
