Commit message: Remove redundant meshes from sensors_description [ci skip]

File: pandora_models/pandora_robots_description/urdf/woody/links/base_link.urdf.xacro (robot description, xacro)
@@ -66,5 +66,7 @@
     </joint>
     <link name="raspberry" >
-      <xacro:solid_cuboid_inertial mass="0.062" width="0.070" height="0.025" depth="0.095" />
+      <xacro:solid_cuboid_inertial mass="0.062" x="0.095" y="0.070" z="0.025" >
+        <xacro:default_origin />
+      </xacro:solid_cuboid_inertial>
     </link>
     <joint name="raspberry_joint"
@@ -76,5 +78,7 @@
     </joint>
     <link name="arm" >
-      <xacro:solid_cuboid_inertial mass="0.050" width="0.064" height="0.03" depth="0.104" />
+      <xacro:solid_cuboid_inertial mass="0.050" x="0.064" y="0.104" z="0.030" >
+        <xacro:default_origin />
+      </xacro:solid_cuboid_inertial>
     </link>
     <joint name="arm_joint"
@@ -181,5 +185,7 @@
     </joint>
     <link name="axis" >
-      <xacro:solid_cylinder_inertial mass="0.446" radius="0.03" height="0.267" />
+      <xacro:solid_cylinder_inertial mass="0.446" radius="0.03" height="0.267" >
+        <xacro:default_origin />
+      </xacro:solid_cylinder_inertial>
     </link>
     <joint name="axis_joint"
@@ -191,5 +197,7 @@
     </joint>
     <link name="imu" >
-      <xacro:solid_cuboid_inertial mass="0.05" width="0.045" height="0.024" depth="0.057" />
+      <xacro:solid_cuboid_inertial mass="0.05" x="0.057" y="0.045" z="0.024" >
+        <xacro:default_origin />
+      </xacro:solid_cuboid_inertial>
     </link>/
     <joint name="imu_joint"

File: pandora_models/pandora_robots_description/urdf/woody/properties/defaults.xacro (robot description, xacro)
@@ -29,9 +29,23 @@
   </xacro:macro>
   <!-- 3D Inertial Objects ################################################ -->
+  <xacro:macro name="point_mass_inertial" >
+    <inertial>
+      <origin xyz="0.0 0.0 0.0" />
+      <mass value="0.001" />
+      <inertia ixx="1.0E-6"
+               ixy="0"
+               ixz="0"
+               iyy="1.0E-6"
+               iyz="0"
+               izz="1.0E-6" />
+    </inertial>
+  </xacro:macro>
   <xacro:macro name="solid_sphere_inertial"
-               params="mass radius" >
+               params="mass
+                       radius
+                       *origin" >
     <inertial>
+      <xacro:insert_block name="origin" />
       <mass value="${mass}" />
-      <xacro:default_origin />
       <inertia ixx="${ ( 2 / 5 ) * mass * ( radius * radius ) }"
                ixy="0.0"
@@ -43,21 +57,28 @@
   </xacro:macro>
   <xacro:macro name="solid_cuboid_inertial"
-               params="mass width height depth" >
+               params="mass
+                       x
+                       y
+                       z
+                       *origin" >
     <inertial>
+      <xacro:insert_block name="origin" />
       <mass value="${mass}" />
-      <xacro:default_origin />
-      <inertia ixx="${ ( 1 / 12 ) * mass * ( ( height * height ) + ( depth * depth ) ) }"
+      <inertia ixx="${ ( 1 / 12 ) * mass * ( ( y * y ) + ( z * z ) ) }"
                ixy="0.0"
                ixz="0.0"
-               iyy="${ ( 1 / 12 ) * mass * ( ( width * width ) + ( depth * depth ) ) }"
+               iyy="${ ( 1 / 12 ) * mass * ( ( x * x ) + ( z * z ) ) }"
                iyz="0.0"
-               izz="${ ( 1 / 12 ) * mass * ( ( width * width ) + ( height * height ) ) }" />
+               izz="${ ( 1 / 12 ) * mass * ( ( x * x ) + ( y * y ) ) }" />
     </inertial>
   </xacro:macro>
   <xacro:macro name="solid_cylinder_inertial"
-               params="mass radius height" >
+               params="mass
+                       radius
+                       height
+                       *origin" >
     <inertial>
+      <xacro:insert_block name="origin" />
       <mass value="${mass}" />
-      <xacro:default_origin />
       <inertia ixx="${ ( 1 / 12 ) * mass * ( 3 * ( radius * radius ) + ( height * height ) ) }"
                ixy="0.0"

File: pandora_models/pandora_robots_description/urdf/woody/sensors/co2_sensor.xacro (robot description, xacro)
@@ -3,6 +3,6 @@
   <xacro:include filename="$(find pandora_sensors_description)/urdf/co2.urdf.xacro" />
   <xacro:macro name="co2_sensor" >
-    <xacro:co2_caster parent="kinect_main_link" >
-      <origin xyz="0.0173 -0.0595 0.022"
+    <xacro:co2_caster parent="kinect_link" >
+      <origin xyz="0.0173 -0.0595 0.0"
               rpy="${zero}" />
     </xacro:co2_caster>

File: pandora_models/pandora_robots_description/urdf/woody/sensors/flir_sensor.xacro (robot description, xacro)
@@ -3,6 +3,6 @@
   <xacro:include filename="$(find pandora_sensors_description)/urdf/flir.urdf.xacro" />
   <xacro:macro name="flir_sensor" >
-    <xacro:flir_caster parent="kinect_main_link" >
-      <origin xyz="0.0173 0.0747 0.022"
+    <xacro:flir_caster parent="kinect_link" >
+      <origin xyz="0.0173 0.0747 0.0"
               rpy="0 0 0" />
     </xacro:flir_caster>

File: pandora_models/pandora_robots_description/urdf/woody/sensors/kinect_sensor.xacro (robot description, xacro)
@@ -10,5 +10,5 @@
                          yaw_min_limit="${kinect_yaw_joint_min_limit}"
                          yaw_max_limit="${kinect_yaw_joint_max_limit}" >
-      <origin xyz="0.08085 0.02998 0.26749"
+      <origin xyz="0.11999 0.031 0.25781"
               rpy="0.0 0.0 0.0" />
     </xacro:kinect_caster>

File: pandora_models/pandora_robots_description/urdf/woody/sensors/laser_sensor.xacro (robot description, xacro)
@@ -5,11 +5,11 @@
                params="fixed" >
     <xacro:laser_caster parent="base_link"
-                         fixed="${fixed}"
-                         roll_min_limit="${laser_roll_joint_min_limit}"
-                         roll_max_limit="${laser_roll_joint_max_limit}"
-                         pitch_min_limit="${laser_pitch_joint_min_limit}"
-                         pitch_max_limit="${laser_pitch_joint_max_limit}" >
-      <origin xyz="0.2185 -0.00219 0.12885"
-              rpy="${zero}" />
+                        fixed="${fixed}"
+                        roll_min_limit="${laser_roll_joint_min_limit}"
+                        roll_max_limit="${laser_roll_joint_max_limit}"
+                        pitch_min_limit="${laser_pitch_joint_min_limit}"
+                        pitch_max_limit="${laser_pitch_joint_max_limit}" >
+      <origin xyz="0.19015 -0.00248 0.12722"
+              rpy="0.0 0.0 0.035" /> <!-- yaw offset -->
     </xacro:laser_caster>
   </xacro:macro>

File: pandora_models/pandora_robots_description/urdf/woody/sensors/microphone_sensor.xacro (robot description, xacro)
@@ -3,5 +3,5 @@
   <xacro:include filename="$(find pandora_sensors_description)/urdf/microphone.urdf.xacro" />
   <xacro:macro name="microphone_sensor" >
-    <xacro:microphone_caster parent="linear_head_main_link" >
+    <xacro:microphone_caster parent="kinect_link" >
       <origin xyz="-0.02175 -0.0374 0.09643"
               rpy="${zero}" />

File: pandora_models/pandora_robots_description/urdf/woody/sensors/thermal_sensor.xacro (robot description, xacro)
@@ -3,7 +3,7 @@
   <xacro:include filename="$(find pandora_sensors_description)/urdf/thermal.urdf.xacro" />
   <xacro:macro name="thermal_sensor" >
-    <xacro:thermal_caster parent="kinect_main_link"
+    <xacro:thermal_caster parent="kinect_link"
                           prefix_y="middle" >
-      <origin xyz="0.0173 0.0949 0.022"
+      <origin xyz="0.0173 0.0949 0.0"
               rpy="0 0 0" />
     </xacro:thermal_caster>
