Commit message: Remove redundant meshes from sensors_description [ci skip]

File: pandora_models/pandora_sensors_description/urdf/kinect.urdf.xacro (robot description, xacro)
@@ -1,5 +1,6 @@
 <?xml version="1.0" ?>
 <robot xmlns:xacro="http://ros.org/wiki/xacro" >
-<!-- ###################################################################### -->
+  <xacro:include filename="$(find pandora_robots_description)/urdf/woody/properties/constants.xacro" />
+  <xacro:include filename="$(find pandora_robots_description)/urdf/woody/properties/defaults.xacro" />
   <xacro:macro name="kinect_caster"
                params="parent
@@ -10,269 +11,110 @@
                        yaw_max_limit
                        *origin" >
-    <!-- ################################################################## -->
-    <link name="kinect_servo_link" >
-      <inertial>
-        <!-- ============================================================== -->
-        <origin xyz="0.00754 0.0 0.00124" />
-        <!-- ============================================================== -->
-        <mass value="0.005" /><!--FIXME-->
-        <!-- ============================================================== -->
-        <inertia ixx="1.0E-6"
-                 ixy="0"
-                 ixz="0"
-                 iyy="1.0E-6"
-                 iyz="0"
-                 izz="1.0E-6" /><!--FIXME-->
-        <!-- ============================================================== -->
-      </inertial>
+    <!-- Links ############################################################ -->
+    <link name="kinect_yaw_servo_link" >
+      <xacro:solid_cuboid_inertial mass="0.055" x="0.050" y="0.032" z="0.049" >
+        <origin xyz="-0.01316 0.00002 0.00093" />
+      </xacro:solid_cuboid_inertial>
       <visual>
-        <!-- ============================================================== -->
-        <origin xyz="-0.01593 0.0 0.0"
-                rpy="0.0 0.0 0.0" />
-        <!-- ============================================================== -->
         <geometry>
-          <mesh filename="package://pandora_sensors_description/meshes/laser/pitch_servo_motor.dae" />
+          <mesh filename="package://pandora_sensors_description/meshes/kinect/yaw_servo_motor.dae" />
         </geometry>
-        <!-- ============================================================== -->
       </visual>
       <collision>
-        <!-- ============================================================== -->
-        <origin xyz="0.00754 0.0 0.00124"
-                rpy="0 0 0" />
-        <!-- ============================================================== -->
+        <origin xyz="-0.0135 0.0 -0.0028" />
         <geometry>
-          <box size="0.050 0.032 0.041" />
+          <box size="0.050 0.032 0.049" />
         </geometry>
-        <!-- ============================================================== -->
       </collision>
     </link>
-    <!-- ################################################################## -->
-    <link name="kinect_base_link" >
-      <inertial>
-        <!-- ============================================================== -->
-        <origin xyz="0.03416 0.0 0.01146" />
-        <!-- ============================================================== -->
-        <mass value="0.005" /><!--FIXME-->
-        <!-- ============================================================== -->
-        <inertia ixx="1.0E-6"
-                 ixy="0"
-                 ixz="0"
-                 iyy="1.0E-6"
-                 iyz="0"
-                 izz="1.0E-6" /><!--FIXME-->
-        <!-- ============================================================== -->
-      </inertial>
+    <link name="kinect_pitch_servo_link" >
+      <xacro:solid_cuboid_inertial mass="0.063" x="0.043" y="0.041" z="0.070" >
+        <origin xyz="0.0001 0.00217 -0.01699" />
+      </xacro:solid_cuboid_inertial>
       <visual>
-        <!-- ============================================================== -->
-        <origin xyz="0 0 0"
-                rpy="0 0 0" />
-        <!-- ============================================================== -->
         <geometry>
-          <mesh filename="package://pandora_sensors_description/meshes/kinect/base.dae" />
+          <mesh filename="package://pandora_sensors_description/meshes/kinect/pitch_servo_motor.dae" />
         </geometry>
-        <!-- ============================================================== -->
       </visual>
       <collision>
-        <!-- ============================================================== -->
-        <origin xyz="0.02131 0.0 0.01992"
-                rpy="0 0 0" />
-        <!-- ============================================================== -->
+        <origin xyz="0.0055 0.0 -0.0405" />
         <geometry>
-          <box size="0.07 0.055 0.04" />
+          <box size="0.043 0.041 0.104" />
         </geometry>
-        <!-- ============================================================== -->
       </collision>
     </link>
-    <!-- ################################################################## -->
-    <link name="kinect_main_link" >
-      <inertial>
-        <!-- ============================================================== -->
-        <origin xyz="0.00052 0.00048 0.02055" />
-        <!-- ============================================================== -->
-        <mass value="0.226796185" />
-        <!-- ============================================================== -->
-        <inertia ixx="1.4641E-3"
-                 ixy="0.0"
-                 ixz="0.0"
-                 iyy="9.2532E-5"
-                 iyz="0.0"
-                 izz="1.5077E-3" />
-        <!-- ============================================================== -->
-      </inertial>
+    <link name="kinect_platform_link" >
+      <xacro:solid_cuboid_inertial mass="0.070" x="0.100" y="0.120" z="0.017" >
+        <origin xyz="0.00926 -0.00059 -0.00362" />
+      </xacro:solid_cuboid_inertial>
       <visual>
-        <!-- ============================================================== -->
-        <origin xyz="0 0 0"
+        <geometry>
+          <mesh filename="package://pandora_sensors_description/meshes/kinect/platform.dae" />
+        </geometry>
+      </visual>
+      <collision>
+        <origin xyz="0.012 -0.00101 -0.019"
                 rpy="0 0 0" />
-        <!-- ============================================================== -->
+        <geometry>
+          <box size="0.100 0.120 0.041" />
+        </geometry>
+      </collision>
+    </link>
+    <link name="kinect_link" >
+      <xacro:solid_cuboid_inertial mass="0.2268" x="0.036" y="0.180" z="0.025" >
+        <origin xyz="0.0000013 0.0 0.0000014" />
+      </xacro:solid_cuboid_inertial>
+      <visual>
         <geometry>
           <mesh filename="package://pandora_sensors_description/meshes/kinect/asus_xtion_pro.dae" />
         </geometry>
-        <!-- ============================================================== -->
       </visual>
       <collision>
-        <!-- ============================================================== -->
-        <origin xyz="0.0 0.0 0.01342"
+        <origin xyz="-0.00075 -0.00048 0.00016"
                 rpy="0 0 0" />
-        <!-- ============================================================== -->
         <geometry>
-          <box size="0.037 0.18 0.042" />
+          <box size="0.036 0.180 0.025" />
         </geometry>
-        <!-- ============================================================== -->
       </collision>
     </link>
-    <!-- ################################################################## -->
     <link name="kinect_frame" >
-      <inertial>
-        <!-- ============================================================== -->
-        <origin xyz="0.0 0.0 0.0" />
-        <!-- ============================================================== -->
-        <mass value="0.005" /><!--FIXME-->
-        <!-- ============================================================== -->
-        <inertia ixx="1.0E-6"
-                 ixy="0"
-                 ixz="0"
-                 iyy="1.0E-6"
-                 iyz="0"
-                 izz="1.0E-6" /><!--FIXME-->
-        <!-- ============================================================== -->
-      </inertial>
+      <xacro:point_mass_inertial />
     </link>
-    <!-- ################################################################## -->
     <link name="kinect_optical_frame" >
-      <inertial>
-        <!-- ============================================================== -->
-        <origin xyz="0.0 0.0 0.0" />
-        <!-- ============================================================== -->
-        <mass value="0.005" /><!--FIXME-->
-        <!-- ============================================================== -->
-        <inertia ixx="1.0E-6"
-                 ixy="0"
-                 ixz="0"
-                 iyy="1.0E-6"
-                 iyz="0"
-                 izz="1.0E-6" /><!--FIXME-->
-        <!-- ============================================================== -->
-      </inertial>
+      <xacro:point_mass_inertial />
     </link>
-    <!-- ################################################################## -->
     <link name="kinect_depth_frame" >
-      <inertial>
-        <!-- ============================================================== -->
-        <origin xyz="0.0 0.0 0.0" />
-        <!-- ============================================================== -->
-        <mass value="0.005" /><!--FIXME-->
-        <!-- ============================================================== -->
-        <inertia ixx="1.0E-6"
-                 ixy="0"
-                 ixz="0"
-                 iyy="1.0E-6"
-                 iyz="0"
-                 izz="1.0E-6" /><!--FIXME-->
-        <!-- ============================================================== -->
-      </inertial>
+      <xacro:point_mass_inertial />
     </link>
-    <!-- ################################################################## -->
     <link name="kinect_depth_optical_frame" >
-      <inertial>
-        <!-- ============================================================== -->
-        <origin xyz="0.0 0.0 0.0" />
-        <!-- ============================================================== -->
-        <mass value="0.005" /><!--FIXME-->
-        <!-- ============================================================== -->
-        <inertia ixx="1.0E-6"
-                 ixy="0"
-                 ixz="0"
-                 iyy="1.0E-6"
-                 iyz="0"
-                 izz="1.0E-6" /><!--FIXME-->
-        <!-- ============================================================== -->
-      </inertial>
+      <xacro:point_mass_inertial />
     </link>
-    <!-- ################################################################## -->
     <link name="kinect_rgb_frame" >
-      <inertial>
-        <!-- ============================================================== -->
-        <origin xyz="0.0 0.0 0.0" />
-        <!-- ============================================================== -->
-        <mass value="0.005" /><!--FIXME-->
-        <!-- ============================================================== -->
-        <inertia ixx="1.0E-6"
-                 ixy="0"
-                 ixz="0"
-                 iyy="1.0E-6"
-                 iyz="0"
-                 izz="1.0E-6" /><!--FIXME-->
-        <!-- ============================================================== -->
-      </inertial>
+      <xacro:point_mass_inertial />
     </link>
-    <!-- ################################################################## -->
     <link name="kinect_rgb_optical_frame" >
-      <inertial>
-        <!-- ============================================================== -->
-        <origin xyz="0.0 0.0 0.0" />
-        <!-- ============================================================== -->
-        <mass value="0.005" /><!--FIXME-->
-        <!-- ============================================================== -->
-        <inertia ixx="1.0E-6"
-                 ixy="0"
-                 ixz="0"
-                 iyy="1.0E-6"
-                 iyz="0"
-                 izz="1.0E-6" /><!--FIXME-->
-        <!-- ============================================================== -->
-      </inertial>
+      <xacro:point_mass_inertial />
     </link>
-    <!-- Pitch Joint #######################################################-->
-    <xacro:if value="${fixed}" >
-      <joint name="kinect_pitch_joint"
-             type="fixed" >
-        <!-- ============================================================== -->
-        <parent link="${parent}" />
-        <child link="kinect_servo_link" />
-        <!-- ============================================================== -->
-        <xacro:insert_block name="origin" />
-        <!-- ============================================================== -->
-      </joint>
-    </xacro:if>
-    <xacro:unless value="${fixed}" >
-      <joint name="kinect_pitch_joint"
-             type="revolute" >
-        <!-- ============================================================== -->
-        <parent link="${parent}" />
-        <child link="kinect_servo_link" />
-        <!-- ============================================================== -->
-        <xacro:insert_block name="origin" />
-        <!-- ============================================================== -->
-        <axis xyz="0 1 0" />
-        <!-- ============================================================== -->
-        <!-- <calibration rising="0.0"
-                          falling="0.0" /> -->
-        <!-- ============================================================== -->
-        <!-- <dynamics damping="0.0"
-                       friction="0.0" /> -->
-        <!-- ============================================================== -->
-        <limit lower="${pitch_min_limit}"
-               upper="${pitch_max_limit}"
-               effort="50"
-               velocity="50.0" />
-        <!-- ============================================================== -->
-        <!-- <safety_controller soft_lower_limit="0.0"
-                                soft_upper_limit="0.0"
-                                k_position="0.0"
-                                k_velocity="0.0" /> -->
-        <!-- ============================================================== -->
-      </joint>
-    </xacro:unless>
-    <!-- Yaw Joint #########################################################-->
+    <!-- Joints ########################################################### -->
+    <joint name="kinect_servo_base_joint"
+           type="fixed" >
+      <parent link="${parent}" />
+      <child link="kinect_yaw_servo_link" />
+      <xacro:insert_block name="origin" />
+    </joint>
     <xacro:if value="${fixed}" >
       <joint name="kinect_yaw_joint"
              type="fixed" >
-        <!-- ============================================================== -->
-        <parent link="kinect_servo_link" />
-        <child link="kinect_base_link" />
-        <!-- ============================================================== -->
-        <origin xyz="0.02107 0.0 0.021"
+        <parent link="kinect_yaw_servo_link" />
+        <child link="kinect_pitch_servo_link" />
+        <origin xyz="0.0 0.0 0.06749"
                 rpy="0.0 0.0 0.0" />
-        <!-- ============================================================== -->
+      </joint>
+      <joint name="kinect_pitch_joint"
+             type="fixed" >
+        <parent link="kinect_pitch_servo_link" />
+        <child link="kinect_platform_link" />
+        <origin xyz="0.0 0.0 0.02852"
+                rpy="0.0 0.0 0.0" />
       </joint>
     </xacro:if>
@@ -280,107 +122,77 @@
       <joint name="kinect_yaw_joint"
              type="revolute" >
-        <!-- ============================================================== -->
-        <parent link="kinect_servo_link" />
-        <child link="kinect_base_link" />
-        <!-- ============================================================== -->
-        <origin xyz="0.02107 0.0 0.021"
+        <parent link="kinect_yaw_servo_link" />
+        <child link="kinect_pitch_servo_link" />
+        <origin xyz="0.0 0.0 0.06749"
                 rpy="0.0 0.0 0.0" />
-        <!-- ============================================================== -->
         <axis xyz="0 0 1" />
-        <!-- ============================================================== -->
-        <!-- <calibration rising="0.0"
-                          falling="0.0" /> -->
-        <!-- ============================================================== -->
-        <!-- <dynamics damping="0.0"
-                       friction="0.0" /> -->
-        <!-- ============================================================== -->
         <limit lower="${yaw_min_limit}"
                upper="${yaw_max_limit}"
                effort="50"
                velocity="50.0" />
-        <!-- ============================================================== -->
-        <!-- <safety_controller soft_lower_limit="0.0"
-                                soft_upper_limit="0.0"
-                                k_position="0.0"
-                                k_velocity="0.0" /> -->
-        <!-- ============================================================== -->
+      </joint>
+      <joint name="kinect_pitch_joint"
+             type="revolute" >
+        <parent link="kinect_pitch_servo_link" />
+        <child link="kinect_platform_link" />
+        <origin xyz="0.0 0.0 0.02852"
+                rpy="0.0 0.0 0.0" />
+        <axis xyz="0 1 0" />
+        <limit lower="${pitch_min_limit}"
+               upper="${pitch_max_limit}"
+               effort="50"
+               velocity="50.0" />
       </joint>
     </xacro:unless>
-    <!-- Base Joint ########################################################-->
-    <joint name="kinect_base_joint"
+    <joint name="kinect_platform_joint"
            type="fixed" >
-      <!-- ================================================================ -->
-      <parent link="kinect_base_link" />
-      <child link="kinect_main_link" />
-      <!-- ================================================================ -->
-      <origin xyz="0.04274 0.0 0.03142"
+      <parent link="kinect_platform_link" />
+      <child link="kinect_link" />
+      <origin xyz="0.03261 -0.00101 0.01409"
               rpy="0.0 0.0 0.0" />
-      <!-- ================================================================ -->
     </joint>
-    <!-- Camera Joint ##################################################### -->
+    <!-- Frames ########################################################### -->
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