Commit message: Remove redundant meshes from sensors_description [ci skip]

File: pandora_models/pandora_sensors_description/urdf/laser.urdf.xacro (robot description, xacro)
@@ -1,5 +1,6 @@
 <?xml version="1.0" ?>
 <robot xmlns:xacro="http://ros.org/wiki/xacro" >
-<!-- ###################################################################### -->
+  <xacro:include filename="$(find pandora_robots_description)/urdf/woody/properties/constants.xacro" />
+  <xacro:include filename="$(find pandora_robots_description)/urdf/woody/properties/defaults.xacro" />
   <xacro:macro name="laser_caster"
                params="parent
@@ -10,105 +11,80 @@
                        pitch_max_limit
                        *origin" >
-    <!-- ################################################################## -->
-    <link name="laser_servo_link" >
-      <inertial>
-        <!-- ============================================================== -->
-        <origin xyz="0.013 0.0 0.00951" />
-        <!-- ============================================================== -->
-        <mass value="0.005" /><!--FIXME-->
-        <!-- ============================================================== -->
-        <inertia ixx="1.0E-6"
-                 ixy="0"
-                 ixz="0"
-                 iyy="1.0E-6"
-                 iyz="0"
-                 izz="1.0E-6" /><!--FIXME-->
-        <!-- ============================================================== -->
-      </inertial>
+    <!-- Links ############################################################ -->
+    <link name="laser_roll_servo_link" >
+      <xacro:solid_cuboid_inertial mass="0.057" x="0.041" y="0.050" z="0.035" >
+        <origin xyz="0.00234 0.01566 -0.0002" />
+      </xacro:solid_cuboid_inertial>
       <visual>
-        <!-- ============================================================== -->
-        <origin xyz="0 0 0"
+        <geometry>
+          <mesh filename="package://pandora_sensors_description/meshes/laser/roll_servo_motor.dae" />
+        </geometry>
+      </visual>
+      <collision>
+        <origin xyz="0.00165 0.0135 -0.0015"
                 rpy="0 0 0" />
-        <!-- ============================================================== -->
+        <geometry>
+          <box size="0.041 0.050 0.035" />
+        </geometry>
+      </collision>
+    </link>
+    <link name="laser_pitch_servo_link" >
+      <xacro:solid_cuboid_inertial mass="0.057" x="0.035" y="0.041" z="0.050" >
+        <origin xyz="-0.00022 0.00223 0.00708" />
+      </xacro:solid_cuboid_inertial>
+      <visual>
         <geometry>
           <mesh filename="package://pandora_sensors_description/meshes/laser/pitch_servo_motor.dae" />
         </geometry>
-        <!-- ============================================================== -->
       </visual>
       <collision>
-        <!-- ============================================================== -->
-        <origin xyz="0.01285 0.00018 0.00959"
+        <origin xyz="-0.00149 0.0 0.0093"
                 rpy="0 0 0" />
-        <!-- ============================================================== -->
         <geometry>
-          <box size="0.032 0.038 0.050" />
+          <box size="0.035 0.041 0.050" />
         </geometry>
-        <!-- ============================================================== -->
       </collision>
     </link>
-    <!-- ################################################################## -->
     <link name="laser_main_link" >
-      <inertial>
-        <!-- ============================================================== -->
-        <origin xyz="0.0 0.0 0.06" />
-        <!-- ============================================================== -->
-        <mass value="0.16" />
-        <!-- ============================================================== -->
-        <inertia ixx="0.0002632"
-                 ixy="0"
-                 ixz="0"
-                 iyy="0.0002632"
-                 iyz="0"
-                 izz="0.000162" />
-        <!-- ============================================================== -->
-      </inertial>
+      <xacro:solid_cuboid_inertial mass="0.160" x="0.048" y="0.051" z="0.80" >
+        <origin xyz="0.00041 -0.00007 0.04539" />
+      </xacro:solid_cuboid_inertial>
       <visual>
-        <!-- ============================================================== -->
-        <origin xyz="0 0 0"
-                rpy="0 0 0" />
-        <!-- ============================================================== -->
         <geometry>
           <mesh filename="package://pandora_sensors_description/meshes/laser/hokuyo_urg_04lx.dae" />
         </geometry>
-        <!-- ============================================================== -->
       </visual>
       <collision>
-        <!-- ============================================================== -->
-        <origin xyz="0 0 0.04822"
+        <origin xyz="0.00078 -0.0001 0.04595"
                 rpy="0 0 0" />
-        <!-- ============================================================== -->
         <geometry>
-          <box size="0.050 0.050 0.114" />
+          <box size="0.048 0.051 0.114" />
         </geometry>
-        <!-- ============================================================== -->
       </collision>
     </link>
-    <!-- ################################################################## -->
     <link name="laser_link" >
-      <inertial>
-        <!-- ============================================================== -->
-        <origin xyz="0.0 0.0 0.0" />
-        <!-- ============================================================== -->
-        <mass value="0.005" /><!--FIXME-->
-        <!-- ============================================================== -->
-        <inertia ixx="1.0E-6"
-                 ixy="0"
-                 ixz="0"
-                 iyy="1.0E-6"
-                 iyz="0"
-                 izz="1.0E-6" /><!--FIXME-->
-        <!-- ============================================================== -->
-      </inertial>
+      <xacro:point_mass_inertial />
     </link>
-    <!-- Roll Joint ####################################################### -->
+    <!-- Joints ########################################################### -->
+    <joint name="laser_servo_base_joint"
+           type="fixed" >
+      <parent link="${parent}" />
+      <child link="laser_roll_servo_link" />
+      <xacro:insert_block name="origin" />
+    </joint>
     <xacro:if value="${fixed}" >
       <joint name="laser_roll_joint"
              type="fixed" >
-        <!-- ============================================================== -->
-        <parent link="${parent}" />
-        <child link="laser_servo_link" />
-        <!-- ============================================================== -->
-        <xacro:insert_block name="origin" />
-        <!-- ============================================================== -->
+        <parent link="laser_roll_servo_link" />
+        <child link="laser_pitch_servo_link" />
+        <origin xyz="0.03999 0.0 0.0"
+                rpy="0 0 0" />
+      </joint>
+      <joint name="laser_pitch_joint"
+             type="fixed" >
+        <parent link="laser_pitch_servo_link" />
+        <child link="laser_main_link" />
+        <origin xyz="0.0 0.0 0.02276"
+                rpy="0 0 0" />
       </joint>
     </xacro:if>
@@ -116,86 +92,34 @@
       <joint name="laser_roll_joint"
              type="revolute" >
-        <!-- ============================================================== -->
-        <parent link="${parent}" />
-        <child link="laser_servo_link" />
-        <!-- ============================================================== -->
-        <xacro:insert_block name="origin" />
-        <!-- ============================================================== -->
+        <parent link="laser_roll_servo_link" />
+        <child link="laser_pitch_servo_link" />
+        <origin xyz="0.03999 0.0 0.0"
+                rpy="0 0 0" />
         <axis xyz="1 0 0" />
-        <!-- ============================================================== -->
-        <!-- <calibration rising="0.0"
-                          falling="0.0" /> -->
-        <!-- ============================================================== -->
-        <!-- <dynamics damping="0.0"
-                       friction="0.0" /> -->
-        <!-- ============================================================== -->
         <limit lower="${roll_min_limit}"
                upper="${roll_max_limit}"
                effort="50"
                velocity="50.0" />
-        <!-- ============================================================== -->
-        <!-- <safety_controller soft_lower_limit="0.0"
-                                soft_upper_limit="0.0"
-                                k_position="0.0"
-                                k_velocity="0.0" /> -->
-        <!-- ============================================================== -->
       </joint>
-    </xacro:unless>
-    <!-- Pitch Joint ###################################################### -->
-    <xacro:if value="${fixed}" >
-      <joint name="laser_pitch_joint"
-             type="fixed" >
-        <!-- ============================================================== -->
-        <parent link="laser_servo_link" />
-        <child link="laser_main_link" />
-        <!-- ============================================================== -->
-        <origin xyz="0.013 0.0 0.02301"
-                rpy="0 0 0" />
-        <!-- ============================================================== -->
-      </joint>
-    </xacro:if>
-    <xacro:unless value="${fixed}" >
       <joint name="laser_pitch_joint"
              type="revolute" >
-        <!-- ============================================================== -->
-        <parent link="laser_servo_link" />
+        <parent link="laser_pitch_servo_link" />
         <child link="laser_main_link" />
-        <!-- ============================================================== -->
-        <origin xyz="0.013 0 0.02301"
+        <origin xyz="0.0 0.0 0.02276"
                 rpy="0 0 0" />
-        <!-- ============================================================== -->
         <axis xyz="0 1 0" />
-        <!-- ============================================================== -->
-        <!-- <calibration rising="0.0"
-                          falling="0.0" /> -->
-        <!-- ============================================================== -->
-        <!-- <dynamics damping="0.0"
-                       friction="0.0" /> -->
-        <!-- ============================================================== -->
         <limit lower="${pitch_min_limit}"
                upper="${pitch_max_limit}"
                effort="50"
                velocity="50.0" />
-        <!-- ============================================================== -->
-        <!-- <safety_controller soft_lower_limit="0.0"
-                                soft_upper_limit="0.0"
-                                k_position="0.0"
-                                k_velocity="0.0" /> -->
-        <!-- ============================================================== -->
       </joint>
     </xacro:unless>
-    <!-- Ray Joint ######################################################## -->
     <joint name="laser_joint"
            type="fixed" >
-      <!-- ================================================================ -->
       <parent link="laser_main_link" />
       <child link="laser_link" />
-      <!-- ================================================================ -->
-      <origin xyz="0.0 0.0 0.08893"
+      <origin xyz="0.0 0.0 0.089"
               rpy="0 0 0" />
-      <!-- ================================================================ -->
     </joint>
-    <!-- ################################################################## -->
   </xacro:macro>
-<!-- ###################################################################### -->
 </robot>

Commit message: Fix sensors' link mass [skip ci]

File: pandora_models/pandora_robots_description/urdf/woody/links/base_link.urdf.xacro (robot description, xacro)
@@ -197,5 +197,5 @@
     </joint>
     <link name="imu" >
-      <xacro:solid_cuboid_inertial mass="0.05" x="0.057" y="0.045" z="0.024" >
+      <xacro:solid_cuboid_inertial mass="0.050" x="0.057" y="0.045" z="0.024" >
         <xacro:default_origin />
       </xacro:solid_cuboid_inertial>

File: pandora_models/pandora_sensors_description/urdf/camera.urdf.xacro (robot description, xacro)
@@ -10,5 +10,5 @@
         <origin xyz="0.00972 0.0 0.04428" />
         <!-- ============================================================== -->
-        <mass value="0.005" />
+        <mass value="0.099" />
         <!-- ============================================================== -->
         <inertia ixx="2.1208E-7"

File: pandora_models/pandora_sensors_description/urdf/co2.urdf.xacro (robot description, xacro)
@@ -10,5 +10,5 @@
         <origin xyz="0.005 0.0 0.0" />
         <!-- ============================================================== -->
-        <mass value="0.005" />
+        <mass value="0.014" />
         <!-- ============================================================== -->
         <inertia ixx="2.1208E-7"

File: pandora_models/pandora_sensors_description/urdf/flir.urdf.xacro (robot description, xacro)
@@ -10,5 +10,5 @@
         <origin xyz="0.00126 0.0 0.0" />
         <!-- ============================================================== -->
-        <mass value="0.005" />
+        <mass value="0.020" />
         <!-- ============================================================== -->
         <inertia ixx="2.1208E-7"

File: pandora_models/pandora_sensors_description/urdf/laser.urdf.xacro (robot description, xacro)
@@ -47,5 +47,5 @@
     </link>
     <link name="laser_main_link" >
-      <xacro:solid_cuboid_inertial mass="0.160" x="0.048" y="0.051" z="0.80" >
+      <xacro:solid_cuboid_inertial mass="0.160" x="0.048" y="0.051" z="0.080" >
         <origin xyz="0.00041 -0.00007 0.04539" />
       </xacro:solid_cuboid_inertial>

File: pandora_models/pandora_sensors_description/urdf/microphone.urdf.xacro (robot description, xacro)
@@ -10,5 +10,5 @@
         <origin xyz="0.01177 0.0 0.0" />
         <!-- ============================================================== -->
-        <mass value="0.005" />
+        <mass value="0.075" />
         <!-- ============================================================== -->
         <inertia ixx="2.1208E-7"

File: pandora_models/pandora_sensors_description/urdf/sonar.urdf.xacro (robot description, xacro)
@@ -10,5 +10,5 @@
         <origin xyz="0.005 0.0 0.0" />
         <!-- ============================================================== -->
-        <mass value="0.010" />
+        <mass value="0.017" />
         <!-- ============================================================== -->
         <inertia ixx="4.2416E-7"
