Commit message: Fix sensor and base inertial [ci skip]

File: pandora_models/pandora_robots_description/woody/urdf/parts/base.urdf.xacro (robot description, xacro)
@@ -3,14 +3,7 @@
   <xacro:macro name="base" >
     <link name="base_link" >
-      <inertial>
-        <origin xyz="-0.00968 -0.00122 0.19369" />
-        <mass value="8.25079" />
-        <inertia ixx="0.112701442"
-                 ixy="-0.000233829"
-                 ixz="-0.014681510"
-                 iyy="0.096589855"
-                 iyz="-0.000177925"
-                 izz="0.083438037" />
-      </inertial>
+      <xacro:solid_cuboid_inertial mass="1.750" x="0.349" y="0.222" z="0.325" >
+        <origin xyz="0.01767 0.00008 0.12635" />
+      </xacro:solid_cuboid_inertial>
       <visual>
         <geometry>
@@ -195,5 +188,5 @@
     </joint>
     <link name="imu" >
-      <xacro:solid_cuboid_inertial mass="0.05" x="0.057" y="0.045" z="0.024" >
+      <xacro:solid_cuboid_inertial mass="0.050" x="0.057" y="0.045" z="0.024" >
         <xacro:default_origin />
       </xacro:solid_cuboid_inertial>

File: pandora_models/pandora_sensors_description/co2/urdf/dynament_gold.urdf.xacro (robot description, xacro)
@@ -5,14 +5,7 @@
     <!-- Links -->
     <link name="co2_link" >
-      <inertial>
+      <xacro:solid_cuboid_inertial mass="0.014" x="0.015" y="0.022" z="0.022" >
         <origin xyz="0.005 0.0 0.0" />
-        <mass value="0.005" />
-        <inertia ixx="2.1208E-7"
-                 ixy="0"
-                 ixz="0"
-                 iyy="4.033E-7"
-                 iyz="0"
-                 izz="2.1208E-7" />
-      </inertial>
+      </xacro:solid_cuboid_inertial>
       <visual>
         <geometry>

File: pandora_models/pandora_sensors_description/laser/urdf/hokuyo_urg_04lx.urdf.xacro (robot description, xacro)
@@ -41,5 +41,5 @@
     </link>
     <link name="laser_main_link" >
-      <xacro:solid_cuboid_inertial mass="0.160" x="0.048" y="0.051" z="0.80" >
+      <xacro:solid_cuboid_inertial mass="0.160" x="0.048" y="0.051" z="0.080" >
         <origin xyz="0.00041 -0.00007 0.04539" />
       </xacro:solid_cuboid_inertial>

File: pandora_models/pandora_sensors_description/laser/urdf/hokuyo_ust_20lx.urdf.xacro (robot description, xacro)
@@ -41,5 +41,5 @@
     </link>
     <link name="laser_main_link" >
-      <xacro:solid_cuboid_inertial mass="0.160" x="0.048" y="0.051" z="0.80" >
+      <xacro:solid_cuboid_inertial mass="0.160" x="0.048" y="0.051" z="0.080" >
         <origin xyz="0.00041 -0.00007 0.04539" />
       </xacro:solid_cuboid_inertial>

File: pandora_models/pandora_sensors_description/microphone/urdf/kinect_array.urdf.xacro (robot description, xacro)
@@ -5,14 +5,7 @@
     <!-- Links -->
     <link name="microphone_link" >
-      <inertial>
+      <xacro:solid_cuboid_inertial mass="0.075" x="0.053" y="0.055" z="0.020" >
         <origin xyz="0.01177 0.0 0.0" />
-        <mass value="0.005" />
-        <inertia ixx="2.1208E-7"
-                 ixy="0"
-                 ixz="0"
-                 iyy="4.033E-7"
-                 iyz="0"
-                 izz="2.1208E-7" />
-      </inertial>
+      </xacro:solid_cuboid_inertial>
       <visual>
         <geometry>

File: pandora_models/pandora_sensors_description/sonar/urdf/devantech_srf05.urdf.xacro (robot description, xacro)
@@ -5,14 +5,7 @@
     <!-- Links -->
     <link name="${name}_sonar_link" >
-      <inertial>
+      <xacro:solid_cuboid_inertial mass="0.017" x="0.015" y="0.044" z="0.022" >
         <origin xyz="0.005 0.0 0.0" />
-        <mass value="0.010" />
-        <inertia ixx="4.2416E-7"
-                 ixy="0.0"
-                 ixz="0.0"
-                 iyy="2.0166E-6"
-                 iyz="0.0"
-                 izz="1.6341E-6" />
-      </inertial>
+      </xacro:solid_cuboid_inertial>
       <visual>
         <geometry>

File: pandora_models/pandora_sensors_description/temperature/urdf/panasonic_grid_eye.urdf.xacro (robot description, xacro)
@@ -5,14 +5,7 @@
     <!-- Links -->
     <link name="${prefix_y}_thermal_link" >
-      <inertial>
+      <xacro:solid_cuboid_inertial mass="0.020" x="0.004" y="0.020" z="0.037" >
         <origin xyz="0.00126 0.0 0.0" />
-        <mass value="0.005" />
-        <inertia ixx="2.1208E-7"
-                 ixy="0"
-                 ixz="0"
-                 iyy="4.033E-7"
-                 iyz="0"
-                 izz="2.1208E-7" />
-      </inertial>
+      </xacro:solid_cuboid_inertial>
       <visual>
         <geometry>

File: pandora_models/pandora_sensors_description/thermal/urdf/flir_lepton.urdf.xacro (robot description, xacro)
@@ -5,14 +5,7 @@
     <!-- Links -->
     <link name="flir_link" >
-      <inertial>
+      <xacro:solid_cuboid_inertial mass="0.020" x="0.004" y="0.020" z="0.037" >
         <origin xyz="0.00126 0.0 0.0" />
-        <mass value="0.005" />
-        <inertia ixx="2.1208E-7"
-                 ixy="0"
-                 ixz="0"
-                 iyy="4.033E-7"
-                 iyz="0"
-                 izz="2.1208E-7" />
-      </inertial>
+      </xacro:solid_cuboid_inertial>
       <visual>
         <geometry>

File: pandora_models/pandora_sensors_description/webcam/urdf/logitech_c310hd.urdf.xacro (robot description, xacro)
@@ -5,14 +5,7 @@
     <!-- Links -->
     <link name="${prefix_y}_camera_link" >
-      <inertial>
+      <xacro:solid_cuboid_inertial mass="0.099" x="0.049" y="0.095" z="0.073" >
         <origin xyz="0.00972 0.0 0.04428" />
-        <mass value="0.005" />
-        <inertia ixx="2.1208E-7"
-                 ixy="0"
-                 ixz="0"
-                 iyy="4.033E-7"
-                 iyz="0"
-                 izz="2.1208E-7" />
-      </inertial>
+      </xacro:solid_cuboid_inertial>
       <visual>
         <geometry>
