Commit message: Fix woody's physics

File: pandora_gazebo/pandora_gazebo_description/woody/urdf_gazebo/sdf_configurations.xacro (robot description, xacro)
@@ -13,6 +13,6 @@
   <xacro:property name="enable_microphone" value="false" />
   <!-- Wheel physics -->
-  <xacro:property name="wheel_mu_1" value="0.75" />
-  <xacro:property name="wheel_mu_2" value="0.75" />
+  <xacro:property name="wheel_mu_1" value="0.9" />
+  <xacro:property name="wheel_mu_2" value="0.85" />
   <xacro:property name="wheel_k_p" value="1000000.0" />
   <xacro:property name="wheel_k_d" value="1.0" />
