Commit message: Change skid steer controller from drive to velocity [ci skip]

File: pandora_gazebo/pandora_gazebo_description/gears/urdf_gazebo/gears.gazebo.xacro (robot description, xacro)
@@ -5,5 +5,5 @@
   <xacro:include filename="$(find pandora_robots_description)/gears/urdf/gears.urdf.xacro" />
   <xacro:include filename="$(find pandora_gazebo_description)/gears/urdf_gazebo/sdf_configurations.xacro" />
-  <xacro:include filename="$(find pandora_gazebo_description)/gears/urdf_gazebo/physics.gazebo.xacro" />
+  <xacro:include filename="$(find pandora_gazebo_description)/gears/urdf_gazebo/references.gazebo.xacro" />
   <xacro:include filename="$(find pandora_gazebo_description)/sdf_elements/sensors/*.gazebo.xacro" />
   <xacro:include filename="$(find pandora_gazebo_description)/sdf_elements/plugins/*.gazebo.xacro" />

File: pandora_gazebo/pandora_gazebo_description/gio/urdf_gazebo/gio.gazebo.xacro (robot description, xacro)
@@ -1,13 +1,11 @@
 <?xml version="1.0"?>
-<robot name="woody"
+<robot name="gio"
        xmlns:xacro="http://ros.org/wiki/xacro" >
   <!-- Import Files -->
-  <xacro:include filename="$(find pandora_robots_description)/woody/urdf/woody.urdf.xacro" />
-  <xacro:include filename="$(find pandora_gazebo_description)/woody/urdf_gazebo/sdf_configurations.xacro" />
-  <xacro:include filename="$(find pandora_gazebo_description)/woody/urdf_gazebo/physics.gazebo.xacro" />
+  <xacro:include filename="$(find pandora_robots_description)/gio/urdf/gio.urdf.xacro" />
+  <xacro:include filename="$(find pandora_gazebo_description)/gio/urdf_gazebo/sdf_configurations.xacro" />
+  <xacro:include filename="$(find pandora_gazebo_description)/gio/urdf_gazebo/references.gazebo.xacro" />
   <xacro:include filename="$(find pandora_gazebo_description)/sdf_elements/sensors/*.gazebo.xacro" />
   <xacro:include filename="$(find pandora_gazebo_description)/sdf_elements/plugins/*.gazebo.xacro" />
-  <!-- Load URDF -->
-  <xacro:woody_urdf />
   <!-- Load gazebo sensors -->
   <xacro:if value="${enable_laser}" >
@@ -38,6 +36,5 @@
   </xacro:if>
   <!-- Load Plugins -->
-  <xacro:gazebo_ros_control interface="pandora_gazebo_interface/WoodyGazeboInterface" />
-  <xacro:pandora_differential />
+  <xacro:gazebo_ros_control interface="pandora_gazebo_interface/GioGazeboInterface" />
   <xacro:pandora_p3d />
   <xacro:if value="$(arg tune)" >

File: pandora_gazebo/pandora_gazebo_description/gio/urdf_gazebo/references.gazebo.xacro (robot description, xacro)
@@ -1,4 +1,51 @@
 <?xml version="1.0" ?>
 <robot xmlns:xacro="http://ros.org/wiki/xacro" >
+  <gazebo>
+    <joint name="differential_left_pin_parallel_joint"
+           type="revolute" >
+      <parent>differential_left_pin_link</parent>
+      <child>left_side_link</child>
+      <pose>0.0 0.0 -0.06533 0.0 0.0 0.0</pose>
+      <axis>
+        <xyz>0 1 0</xyz>
+        <limit>
+          <lower>-0.785</lower>
+          <upper>0.785</upper>
+        </limit>
+        <dynamics>
+          <friction>0</friction>
+          <damping>10</damping>
+        </dynamics>
+      </axis>
+    </joint>
+  </gazebo>
+  <gazebo>
+    <joint name="differential_right_pin_parallel_joint"
+           type="revolute" >
+      <parent>differential_right_pin_link</parent>
+      <child>right_side_link</child>
+      <pose>0.0 0.0 -0.06533 0.0 0.0 0.0</pose>
+      <axis>
+        <xyz>0 1 0</xyz>
+        <limit>
+          <lower>-0.785</lower>
+          <upper>0.785</upper>
+        </limit>
+        <dynamics>
+          <friction>0</friction>
+          <damping>10</damping>
+        </dynamics>
+      </axis>
+    </joint>
+  </gazebo>
+  <gazebo reference="linear_actuator_joint" >
+    <implicitSpringDamper>true</implicitSpringDamper>
+  </gazebo>
+  <gazebo reference="camera_effector_pan_joint" >
+    <implicitSpringDamper>true</implicitSpringDamper>
+  </gazebo>
+  <gazebo reference="camera_effector_tilt_joint" >
+    <implicitSpringDamper>true</implicitSpringDamper>
+  </gazebo>
   <gazebo reference="left_front_wheel_link" >
     <minDepth>${wheel_min_depth}</minDepth>

File: pandora_gazebo/pandora_gazebo_description/sdf_elements/sensors/laser_sensor.gazebo.xacro (robot description, xacro)
@@ -9,6 +9,6 @@
               <samples>683</samples>
               <resolution>1</resolution>
-              <min_angle>-2.26889</min_angle>
-              <max_angle>2.268899</max_angle>
+              <min_angle>-2.00712864</min_angle>
+              <max_angle>2.00712864</max_angle>
             </horizontal>
           </scan>
