Commit message: Fix color of camera_effector's meshes [ci skip]

File: pandora_models/pandora_robots_description/gears/urdf/parts/base.urdf.xacro (robot description, xacro)
@@ -17,5 +17,4 @@
           <mesh filename="package://pandora_robots_description/gears/meshes/base_link.dae" />
         </geometry>
-        <material name="base" />
       </visual>
       <collision>

File: pandora_models/pandora_robots_description/gears/urdf/parts/linear_elevator.urdf.xacro (robot description, xacro)
@@ -17,5 +17,4 @@
           <mesh filename="package://pandora_robots_description/gears/meshes/linear_elevator_link.dae" />
         </geometry>
-        <material name="linear_elevator" />
       </visual>
       <collision>

File: pandora_models/pandora_robots_description/gears/urdf/parts/linear_head.urdf.xacro (robot description, xacro)
@@ -12,5 +12,4 @@
           <mesh filename="package://pandora_robots_description/gears/meshes/servo_motor.dae" />
         </geometry>
-        <material name="linear_head_base" />
       </visual>
       <collision>

File: pandora_models/pandora_robots_description/gears/urdf/parts/side.urdf.xacro (robot description, xacro)
@@ -20,5 +20,4 @@
           <mesh filename="package://pandora_robots_description/gears/meshes/side_link.dae" />
         </geometry>
-        <material name="side" />
       </visual>
       <collision>

File: pandora_models/pandora_robots_description/gears/urdf/parts/wheel.urdf.xacro (robot description, xacro)
@@ -20,5 +20,4 @@
           <mesh filename="package://pandora_robots_description/gears/meshes/wheel_link.dae" />
         </geometry>
-        <material name="wheel" />
       </visual>
       <collision>

File: pandora_models/pandora_robots_description/gio/urdf/parts/base.urdf.xacro (robot description, xacro)
@@ -10,5 +10,4 @@
           <mesh filename="package://pandora_robots_description/gio/meshes/base_link.dae" />
         </geometry>
-        <material name="base" />
       </visual>
       <collision>

File: pandora_models/pandora_robots_description/gio/urdf/parts/side.urdf.xacro (robot description, xacro)
@@ -20,5 +20,4 @@
           <mesh filename="package://pandora_robots_description/gio/meshes/side_link.dae" />
         </geometry>
-        <material name="side" />
       </visual>
       <collision>

File: pandora_models/pandora_robots_description/gio/urdf/parts/wheel.urdf.xacro (robot description, xacro)
@@ -13,5 +13,4 @@
           <mesh filename="package://pandora_robots_description/gio/meshes/wheel_link.dae" />
         </geometry>
-        <material name="wheel" />
       </visual>
       <collision>

File: pandora_models/pandora_urdf_properties/xacro/materials.xacro (robot description, xacro)
@@ -19,12 +19,3 @@
     <color rgba="${192/255} ${192/255} ${192/255} 1.0" />
   </material>
-  <material name="base" >
-    <color rgba="${0/255} ${0/255} ${0/255} 1.0" />
-  </material>
-  <material name="side" >
-    <color rgba="${0/255} ${0/255} ${0/255} 1.0" />
-  </material>
-  <material name="wheel" >
-    <color rgba="${5/255} ${5/255} ${0/255} 1.0" />
-  </material>
 </robot>
