Commit message: Fix camera_effector's macro name and published topic [ci skip]

File: pandora_gazebo/pandora_gazebo_description/sdf_elements/sensors/camera_effector.gazebo.xacro (robot description, xacro)
@@ -1,5 +1,5 @@
 <?xml version="1.0"?>
 <robot xmlns:xacro="http://ros.org/wiki/xacro" >
-  <xacro:macro name="camera_effector" >
+  <xacro:macro name="camera_effector_sensor" >
     <gazebo reference="pi_camera_frame" >
       <sensor name="pi_camera" type="camera" >
@@ -18,5 +18,5 @@
         <plugin name="camera2ros" filename="libgazebo_ros_camera.so" >
           <frameName>pi_camera_optical_frame</frameName>
-          <cameraName>pi_camera</cameraName>
+          <cameraName>rpi2/pi_camera</cameraName>
           <imageTopicName>image</imageTopicName>
         </plugin>
