Commit message: Remove redundant files [ci skip]

File: pandora_gazebo/pandora_gazebo_description/gio/urdf_gazebo/gio.gazebo.xacro (robot description, xacro)
@@ -18,4 +18,7 @@
     <xacro:thermal_sensor />
   </xacro:if>
+  <xacro:if value="${enable_camera_effector}" >
+    <xacro:camera_effector_sensor />
+  </xacro:if>
   <xacro:if value="${enable_webcam}" >
     <xacro:webcam_sensor prefix_y="left" />
@@ -28,7 +31,4 @@
   <xacro:if value="${enable_co2}" >
     <xacro:co2_sensor />
-  </xacro:if>
-  <xacro:if value="${enable_temperature}" >
-    <xacro:temperature_sensor prefix_y="middle" />
   </xacro:if>
   <xacro:if value="${enable_microphone}" >

File: pandora_gazebo/pandora_gazebo_description/gio/urdf_gazebo/sdf_configurations.xacro (robot description, xacro)
@@ -7,8 +7,8 @@
   <xacro:property name="enable_kinect" value="true" />
   <xacro:property name="enable_thermal" value="false" />
+  <xacro:property name="enable_camera_effector" value="true" />
   <xacro:property name="enable_webcam" value="true" />
   <xacro:property name="enable_sonar" value="true" />
   <xacro:property name="enable_co2" value="true" />
-  <xacro:property name="enable_temperature" value="false" />
   <xacro:property name="enable_microphone" value="false" />
   <!-- Wheel physics -->
