Commit message: Change sonar fov

File: pandora_gazebo/pandora_gazebo_description/gio/urdf_gazebo/sdf_configurations.xacro (robot description, xacro)
@@ -13,6 +13,6 @@
   <xacro:property name="enable_microphone" value="false" />
   <!-- Wheel physics -->
-  <xacro:property name="wheel_mu_1" value="0.9" />
-  <xacro:property name="wheel_mu_2" value="0.85" />
+  <xacro:property name="wheel_mu_1" value="0.85" />
+  <xacro:property name="wheel_mu_2" value="0.70" />
   <xacro:property name="wheel_k_p" value="1000000.0" />
   <xacro:property name="wheel_k_d" value="1.0" />

File: pandora_gazebo/pandora_gazebo_description/sdf_elements/sensors/sonar.gazebo.xacro (robot description, xacro)
@@ -9,6 +9,6 @@
               <samples>12</samples>
               <resolution>1</resolution>
-              <min_angle>-0.5235987756</min_angle>
-              <max_angle>0.5235987756</max_angle>
+              <min_angle>-0.07913</min_angle>
+              <max_angle>0.07913</max_angle>
             </horizontal>
             <vertical>
