Commit message: Adjust linear and camera_effector inertial [ci skip]

File: pandora_models/pandora_robots_description/gio/urdf/parts/linear.urdf.xacro (robot description, xacro)
@@ -20,7 +20,15 @@
     </link>
     <link name="linear_actuator_link" >
-      <xacro:solid_cuboid_inertial mass="0.029" x="0.009" y="0.009" z="0.100" >
-        <origin xyz="0.0 0.0 0.05034" />
-      </xacro:solid_cuboid_inertial>
+      <!-- FIXME -->
+      <inertial>
+        <origin xyz="0.017561 0.0109 0.24001" />
+        <mass value="0.92399" />
+        <inertia ixx="0.0097139"
+                 ixy="-0.00039516"
+                 ixz="-0.00086264"
+                 iyy="0.0095873"
+                 iyz="0.0012764"
+                 izz="0.0017829" />
+      </inertial>
       <visual>
         <geometry>

File: pandora_models/pandora_sensors_description/camera_effector/urdf/pi_camera.urdf.xacro (robot description, xacro)
@@ -7,6 +7,7 @@
     <!-- Links -->
     <link name="camera_effector_pan_link" >
-      <xacro:solid_cuboid_inertial mass="0.020" x="0.012" y="0.032" z="0.029" >
-        <origin xyz="0.0 -0.00518 0.01887" />
+      <!-- FIXME -->
+      <xacro:solid_cuboid_inertial mass="0.057" x="0.041" y="0.050" z="0.035" >
+        <origin xyz="0.00234 0.01566 -0.0002" />
       </xacro:solid_cuboid_inertial>
       <visual>
@@ -55,7 +56,15 @@
     </link>
     <link name="pi_camera_platform_link" >
-      <xacro:solid_cuboid_inertial mass="0.005" x="0.011" y="0.050" z="0.030" >
-        <origin xyz="0.0 -0.01085 0.01074" />
-      </xacro:solid_cuboid_inertial>
+      <!-- FIXME -->
+      <inertial>
+        <origin xyz="-0.00329 -0.02726 0.05623" />
+        <mass value="0.16491" />
+        <inertia ixx="0.00030418"
+                 ixy="-1.3735E-05"
+                 ixz="-2.3947E-05"
+                 iyy="0.00015881"
+                 iyz="-7.9817E-06"
+                 izz="0.00024855" />
+      </inertial>
       <visual>
         <geometry>
