Commit message: Change sonar orientation [ci skip]

File: pandora_models/pandora_robots_description/gio/urdf/parts/base.urdf.xacro (robot description, xacro)
@@ -12,20 +12,13 @@
       </visual>
       <collision>
-        <origin xyz="0.02514 0.0 0.14619" />
         <geometry>
-          <box size="0.336 0.225 0.315" />
+          <mesh filename="package://pandora_robots_description/gio/meshes/base_link.stl" />
         </geometry>
       </collision>
     </link>
     <link name="miniitx" >
-      <inertial>
-        <mass value="0.589" />
-        <inertia ixx="0.0014381417"
-                 ixy="0.0"
-                 ixz="0.0"
-                 iyy="0.0019829667"
-                 iyz="0.0"
-                 izz="0.0033818417" />
-      </inertial>
+      <xacro:solid_cuboid_inertial mass="0.589" x="0.17" y="0.17" z="0.04" >
+        <origin xyz="0.0 0.0 0.0" />
+      </xacro:solid_cuboid_inertial>
     </link>
     <joint name="miniitx_joint"
@@ -36,13 +29,7 @@
     </joint>
     <link name="ssd" >
-      <inertial>
-        <mass value="0.078" />
-        <inertia ixx="0.0000325"
-                 ixy="0.0"
-                 ixz="0.0"
-                 iyy="0.00006565"
-                 iyz="0.0"
-                 izz="0.00009685" />
-      </inertial>
+      <xacro:solid_cuboid_inertial mass="0.078" x="0.1" y="0.01" z="0.07" >
+        <origin xyz="0.0 0.0 0.0" />
+      </xacro:solid_cuboid_inertial>
     </link>
     <joint name="ssd_joint"
@@ -78,13 +65,7 @@
     </joint>
     <link name="epos" >
-      <inertial>
-        <mass value="0.136" />
-        <inertia ixx="0.0002266667"
-                 ixy="0.0"
-                 ixz="0.0"
-                 iyy="6.8283E-005"
-                 iyz="0.0"
-                 izz="0.0002858833" />
-      </inertial>
+      <xacro:solid_cuboid_inertial mass="0.136" x="0.075" y="0.14" z="0.04" >
+        <origin xyz="0.0 0.0 0.0" />
+      </xacro:solid_cuboid_inertial>
     </link>
     <joint name="epos_joint"
@@ -95,13 +76,7 @@
     </joint>
     <link name="psu" >
-      <inertial>
-        <mass value="0.178" />
-        <inertia ixx="0.0002241168"
-                 ixy="0.0"
-                 ixz="0.0"
-                 iyy="0.0001828208"
-                 iyz="0.0"
-                 izz="0.0004002627" />
-      </inertial>
+      <xacro:solid_cuboid_inertial mass="0.178" x="0.094" y="0.122" z="0.02" >
+        <origin xyz="0.0 0.0 0.0" />
+      </xacro:solid_cuboid_inertial>
     </link>
     <joint name="psu_joint"
@@ -112,13 +87,7 @@
     </joint>
     <link name="motor_battery" >
-      <inertial>
-        <mass value="0.8" />
-        <inertia ixx="0.0003576"
-                 ixy="0.0"
-                 ixz="0.0"
-                 iyy="0.0016806"
-                 iyz="0.0"
-                 izz="0.0015582" />
-      </inertial>
+      <xacro:solid_cuboid_inertial mass="0.8" x="0.154" y="0.049" z="0.052" >
+        <origin xyz="0.0 0.0 0.0" />
+      </xacro:solid_cuboid_inertial>
     </link>
     <joint name="motor_battery_joint"
@@ -129,13 +98,7 @@
     </joint>
     <link name="pc_battery" >
-      <inertial>
-        <mass value="0.8" />
-        <inertia ixx="0.0003576"
-                 ixy="0.0"
-                 ixz="0.0"
-                 iyy="0.0016806"
-                 iyz="0.0"
-                 izz="0.0015582" />
-      </inertial>
+      <xacro:solid_cuboid_inertial mass="0.8" x="0.154" y="0.049" z="0.052" >
+        <origin xyz="0.0 0.0 0.0" />
+      </xacro:solid_cuboid_inertial>
     </link>
     <joint name="pc_battery_joint"
@@ -145,25 +108,13 @@
       <origin xyz="0.10395 -0.027 0.04822" />
     </joint>
-    <link name="cables" >
-      <inertial>
-        <mass value="0.6" />
-        <inertia ixx="0.00001"
-                 ixy="0.0"
-                 ixz="0.0"
-                 iyy="0.00001"
-                 iyz="0.0"
-                 izz="0.00001" />
-      </inertial>
-    </link>
-    <joint name="cables_joint"
-           type="fixed" >
-      <parent link="base_link" />
-      <child link="cables" />
-      <origin xyz="0.0 0.0 0.1" />
-    </joint>
     <link name="axis" >
       <xacro:solid_cylinder_inertial mass="0.446" radius="0.03" y="0.267" >
         <xacro:default_origin />
       </xacro:solid_cylinder_inertial>
+      <collision>
+        <geometry>
+          <box size="0.057 0.267 0.025" />
+        </geometry>
+      </collision>
     </link>
     <joint name="axis_joint"

File: pandora_models/pandora_robots_description/gio/urdf/sensors/sonar.xacro (robot description, xacro)
@@ -5,6 +5,6 @@
     <xacro:devantech_srf05 name="left"
                            parent="base_link" >
-      <origin xyz="-0.15974 0.11037 0.14973"
-              rpy="0.0 0.0 ${- PI_6 }" />
+      <origin xyz="-0.15974 0.07913 0.14973"
+              rpy="0.0 0.0 0.097651" />
     </xacro:devantech_srf05>
   </xacro:macro>
@@ -12,6 +12,6 @@
     <xacro:devantech_srf05 name="right"
                            parent="base_link" >
-      <origin xyz="-0.15974 -0.11037 0.14973"
-              rpy="0.0 0.0 ${ PI_6 }" />
+      <origin xyz="-0.15974 -0.07913 0.14973"
+              rpy="0.0 0.0 -0.097651" />
     </xacro:devantech_srf05>
   </xacro:macro>
