Commit message: Fix collisions of linear and camera_effector [ci skip]

File: pandora_models/pandora_sensors_description/kinect/urdf/asus_xtion_pro_live.urdf.xacro (robot description, xacro)
@@ -48,8 +48,8 @@
       </visual>
       <collision>
-        <origin xyz="0.012 -0.00101 -0.019"
+        <origin xyz="0.0095 0.0 0.04851"
                 rpy="0 0 0" />
         <geometry>
-          <box size="0.100 0.120 0.041" />
+          <box size="0.096 0.180 0.043" />
         </geometry>
       </collision>
@@ -105,5 +105,5 @@
       <parent link="kinect_platform_link" />
       <child link="kinect_link" />
-      <origin xyz="0.03261 -0.00101 0.04261"
+      <origin xyz="0.01461 -0.00106 0.05011"
               rpy="0.0 0.0 0.0" />
     </joint>

File: pandora_models/pandora_urdf_properties/xacro/defaults.xacro (robot description, xacro)
@@ -28,5 +28,5 @@
              izz="1.0" />
   </xacro:macro>
-  <!-- 3D Inertial Objects ################################################ -->
+  <!-- 3D Inertial Objects  -->
   <xacro:macro name="point_mass_inertial" >
     <inertial>
@@ -69,14 +69,14 @@
   </xacro:macro>
   <xacro:macro name="solid_cylinder_inertial"
-               params="mass radius height *origin" >
+               params="mass radius y *origin" >
     <inertial>
       <xacro:insert_block name="origin" />
       <mass value="${mass}" />
-      <inertia ixx="${(1 / 12) * mass * (3 * (radius * radius) + (height * height))}"
+      <inertia ixx="${(1 / 12) * mass * (3 * (radius * radius) + (y * y))}"
                ixy="0.0"
                ixz="0.0"
-               iyy="${(1 / 12) * mass * (3 * (radius * radius) + (height * height))}"
+               iyy="${(1 / 2) * mass * (radius * radius)}"
                iyz="0.0"
-               izz="${(1 / 2) * mass * (radius * radius)}" />
+               izz="${(1 / 12) * mass * (3 * (radius * radius) + (y * y))}" />
     </inertial>
   </xacro:macro>

Commit message: Fix kinect_platform_link rpy [ci skip]

File: pandora_models/pandora_sensors_description/kinect/urdf/asus_xtion_pro_live.urdf.xacro (robot description, xacro)
@@ -95,4 +95,6 @@
       <parent link="kinect_pitch_servo_link" />
       <child link="kinect_platform_link" />
+      <origin xyz="0.0 0.0 0.0"
+              rpy="0.0 -0.0174 0.0" />
       <axis xyz="0 1 0" />
       <limit lower="${pitch_min_limit}"
@@ -106,5 +108,5 @@
       <child link="kinect_link" />
       <origin xyz="0.01461 -0.00106 0.05011"
-              rpy="0.0 0.0 0.0" />
+              rpy="0.0 0.0674 0.0" />
     </joint>
     <!-- Frames -->

Commit message: Fix kinect_frame position

File: pandora_models/pandora_sensors_description/kinect/urdf/asus_xtion_pro_live.urdf.xacro (robot description, xacro)
@@ -133,5 +133,5 @@
       <parent link="kinect_link" />
       <child link="kinect_frame" />
-      <origin xyz="0.01784 0.0 0.02167"
+      <origin xyz="0.01784 0.0 0.0"
               rpy="0.0 0.0 0.0" />
     </joint>
